File: pcbs/power/power_board.kicad_pcb (KiCad board)
At the start: 2 copper layers, 114 x 137.6 mm, 36 parts, among them J1 PinSocket_1x04_P2.54, J10 MR30PW-M, J11 MR30PW-M, J2 PinSocket_1x04_P2.54, J3 PinSocket_1x04_P2.54, J4 JST_XH_B3B, J5 JST_XH_B3B, J6 XT30PW-F, J7 XT30PW-F, J8 XT30PW-M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

Commit message: Update for CNC
Parts:
- added J12: 12V connection, oxebots_connectors:JST_B2B-XH-A, F.Cu at (72.4, 103.9)
Routing:
- net +12V: track 20.7 -> 51.1 mm
- net V_{ BATT}: track 248.9 -> 223.6 mm
