File: pcbs/power/power_board.kicad_sch (KiCad schematic)
At the start: 31 parts, among them J10 MR30PW-M, J11 MR30PW-M, J12 12V connection, J4 JST_XH_B3B, J5 JST_XH_B3B, J6 XT30PW-F, J7 XT30PW-F, J8 XT30PW-M, J9 MR30PW-M

Commit message: Atualização para versão 10.0 do kicad Condensação do Layout Mudança no circuito V_mon para diminuir impedância de saída Implementação de Circuito "E-Switch" low side Resolução de EDR's no esquemático e PCB
Parts:
- removed C1: 100nF, PCM_Capacitor_THT_AKL:C_Disc_D5.0mm_W2.5mm_P5.00mm, symbol PCM_Capacitor_AKL:C_Generic
- removed D1: 1.5KE30CA, PCM_Diode_THT_AKL:D_DO-201_P12.70mm_Horizontal_TVS, symbol PCM_Diode_TVS_AKL:1.5KE30CA
- removed F1: 30A, oxebots:FUSE_3557-10, symbol 3557-10:3557-10
- removed J12: 12V connection, oxebots_connectors:JST_B2B-XH-A, symbol Connector_Generic:Conn_01x02
- removed J4, J5: JST_XH_B3B, Connector_JST:JST_XH_B3B-XH-A_1x03_P2.50mm_Vertical, symbol Connector_Generic:Conn_01x03
- removed J6, J7: XT30PW-F, oxebots_connectors:AMASS_XT30PW-F, symbol oxebots:XT30PW-F
- removed J8: XT30PW-M, oxebots_connectors:AMASS_XT30PW-M, symbol XT30PW-M:XT30PW-M
- removed TP2: SW_{NO}, TestPoint:TestPoint_Pad_D1.0mm, symbol Connector:TestPoint
- removed TP3: V+, TestPoint:TestPoint_Pad_D2.5mm, symbol Connector:TestPoint
- removed TP4: V^{-}_{no}, TestPoint:TestPoint_Pad_D2.5mm, symbol Connector:TestPoint
- removed TP5: B+, TestPoint:TestPoint_Pad_D2.5mm, symbol Connector:TestPoint
- removed TP6: V-, TestPoint:TestPoint_Pad_D2.5mm, symbol Connector:TestPoint
- removed TP7: P-, Connector_Wire:SolderWirePad_1x01_SMD_5x10mm, symbol Connector:TestPoint
- added C1, C2, C9: 10uF, Capacitor_THT:CP_Radial_D5.0mm_P2.50mm, symbol Device:C
- added C10, C4, C5: 0.01uF, Capacitor_THT:C_Disc_D3.0mm_W1.6mm_P2.50mm, symbol Device:C
- added C11: 220uF, Capacitor_SMD:CP_Elec_8x6.2, symbol Device:C_US
- added C3: 100nF, Capacitor_THT:C_Disc_D3.0mm_W1.6mm_P2.50mm, symbol Device:C
- added C6, C7: 220uF, Capacitor_SMD:CP_Elec_6.3x7.7, symbol Device:C_US
- added C8: 10uF, Capacitor_THT:CP_Radial_D5.0mm_P2.50mm, symbol Device:C_US
- added D1, D2, D8: B340, Diode_SMD:D_SMC, symbol Diode:B340
- added D3: 1N4744A, Diode_THT:D_DO-41_SOD81_P10.16mm_Horizontal, symbol Diode:1N47xxA
- added D4: 1.5KE30CA, Diode_THT:D_DO-201AE_P15.24mm_Horizontal, symbol Diode:1.5KExxCA
- added D5, D6, D7: LED, LED_SMD:LED_0805_2012Metric, symbol Device:LED
- added F1: 30, Fuse:Fuseholder_Blade_Mini_Keystone_3568, symbol Device:Fuse
- added J1: Conn_02x08_Odd_Even, Connector_IDC:IDC-Header_2x08_P2.54mm_Vertical, symbol Connector_Generic:Conn_02x08_Odd_Even
- added J2: XT30PW-F, Connector_AMASS:AMASS_XT30PW-F_1x02_P2.50mm_Horizontal, symbol XT30PW-F:XT30PW-F
- added J3: XT30PW-M, Connector_AMASS:AMASS_XT30PW-M_1x02_P2.50mm_Horizontal, symbol XT30PW-M:XT30PW-M
- added J7: JST_XH_B3B, Connector_JST:JST_XH_B3B-XH-A_1x03_P2.50mm_Vertical, symbol Connector_Generic:Conn_01x03
- added L1, L2, L3: 22uH, Inductor_SMD:L_6.3x6.3_H3, symbol Device:L_Iron
- added Q1: IRFB3205, Package_TO_SOT_THT:TO-220-3_Vertical, symbol Transistor_FET:IRF740
- added R10: 120, Resistor_SMD:R_0805_2012Metric, symbol Device:R_US
- added R11, R12: 1k, Resistor_SMD:R_0805_2012Metric, symbol Device:R_US
- added R13, R6, R7: 10k, Resistor_SMD:R_0805_2012Metric, symbol Device:R_US
- added R3: 2.7k, Resistor_SMD:R_0805_2012Metric, symbol Device:R_US
- added R4: 5.6k, Resistor_SMD:R_0805_2012Metric, symbol Device:R_US
- added R5: 100K, Resistor_THT:R_Axial_DIN0204_L3.6mm_D1.6mm_P5.08mm_Horizontal, symbol Device:R_US
- added R8: 10k, Resistor_THT:R_Axial_DIN0204_L3.6mm_D1.6mm_P5.08mm_Horizontal, symbol Device:R_US
- added R9: 330, Resistor_SMD:R_0805_2012Metric, symbol Device:R_US
- added R_ADJ1, R_ADJ2: 1K, Potentiometer_SMD:Potentiometer_Bourns_3314G_Vertical, symbol Device:R_Potentiometer_Trim_US
- added R_ADJ3: 220, Potentiometer_SMD:Potentiometer_Bourns_3314G_Vertical, symbol Device:R_Potentiometer_Trim_US
- added U1, U2, U3: TPS5430DDA, Package_SO:TI_SO-PowerPAD-8_ThermalVias, symbol Regulator_Switching:TPS5430DDA
- H1, H2, H3: KiLib_Generator (none) -> mounting_hardware/mounting_hole
- J4: renamed from J9; footprint oxebots_connectors:AMASS_MR30PW-M_1x03_P3.50mm_Horizontal -> oxebots:AMASS_MR30PW-M_1x03_P3.50mm_Horizontal
- J5: renamed from J10; footprint oxebots_connectors:AMASS_MR30PW-M_1x03_P3.50mm_Horizontal -> oxebots:AMASS_MR30PW-M_1x03_P3.50mm_Horizontal
- J6: renamed from J11; footprint oxebots_connectors:AMASS_MR30PW-M_1x03_P3.50mm_Horizontal -> oxebots:AMASS_MR30PW-M_1x03_P3.50mm_Horizontal
- R1: value 5.6M -> 56K; footprint PCM_Resistor_THT_AKL:R_Axial_DIN0204_L3.6mm_D1.6mm_P5.08mm_Horizontal -> Resistor_THT:R_Axial_DIN0204_L3.6mm_D1.6mm_P5.08mm_Horizontal; KiLib_Generator (none) -> resistor/THT
- R2: value 220K -> 2.2K; footprint PCM_Resistor_THT_AKL:R_Axial_DIN0204_L3.6mm_D1.6mm_P5.08mm_Horizontal -> Resistor_THT:R_Axial_DIN0204_L3.6mm_D1.6mm_P5.08mm_Horizontal; KiLib_Generator (none) -> resistor/THT
- TP1: value SW+ -> P-
- renumbered TP12 to TP2, TP13 to TP3, TP14 to TP4, TP8 to TP5, TP9 to TP6, TP10 to TP7, TP11 to TP8
Connections:
- net +12V: now also C11.1, J1.7 (Pin_7), L3.2, R12.1, R13.1
- net +3.3V: now also C7.1, J1.9 (Pin_9), L2.2, R10.1, R7.1
- net +5V: now also C6.1, J1.8 (Pin_8), L1.2, R6.1, R9.1
- net B_{6s}: now also F1.1
- net GND: now also C1.2, C11.2, C2.2, C3.2, C6.2, C7.2, C9.2, D1.2 (A), D2.2 (A), D4.2 (A2), D5.1 (K), D6.1 (K), D7.1 (K), D8.2 (A), J1.11 (Pin_11), J1.12 (Pin_12), J1.13 (Pin_13), J1.14 (Pin_14), J1.15 (Pin_15), J1.16 (Pin_16), J2.N, J7.1 (Pin_1), Q1.2 (D), R_ADJ1.2, R_ADJ1.3, R_ADJ2.2, R_ADJ2.3, R_ADJ3.2, R_ADJ3.3, U1.6 (GND), U1.9 (GNDPAD), U2.6 (GND), U2.9 (GNDPAD), U3.6 (GND), U3.9 (GNDPAD)
- net GND_{BMS}: now also TP1.1, C8.2, D3.2 (A), J3.N, Q1.3 (S), R5.2
- net V_{ BATT}: now also C1.1, C2.1, C9.1, D4.1 (A1), F1.2, J1.1 (Pin_1), J1.2 (Pin_2), J1.3 (Pin_3), J1.4 (Pin_4), J1.5 (Pin_5), J1.6 (Pin_6), J2.P, J3.P, J7.3 (Pin_3), U1.7 (VIN), U2.7 (VIN), U3.7 (VIN); no longer TP1.1
- net V_{MON} renamed VMon
- net VMon: now also C3.1, J1.10 (Pin_10)
- new net: C10.2, D8.1 (K), L3.1, U3.8 (PH)
- new net: C10.1, U3.1 (BOOT)
- new net: C8.1, D3.1 (K), Q1.1 (G), R5.1, R8.2
- new net: C4.1, U1.1 (BOOT)
- new net: R3.2, R6.2, U1.4 (VSENSE)
- new net: C4.2, D1.1 (K), L1.1, U1.8 (PH)
- new net: C5.1, U2.1 (BOOT)
- new net: R4.2, R7.2, U2.4 (VSENSE)
- new net: C5.2, D2.1 (K), L2.1, U2.8 (PH)
- new net: R3.1, R_ADJ1.1
- new net: D7.2 (A), R12.2
- new net: R11.1, R_ADJ3.1
- new net: R11.2, R13.2, U3.4 (VSENSE)
- new net: D5.2 (A), R9.2
- new net: D6.2 (A), R10.2
- new net: R4.1, R_ADJ2.1
- new net SW_{NO}: J7.2 (Pin_2), R8.1
- no-connect marks 0 -> 3
Other:
- removed sheet VOLTAGE CONVERTER
- note added: "+12V_ALW_BUCK"
- note added: "+3V3_ALW_BUCK"
- note added: "+5V_ALW_BUCK"
- note added: "Connector for Motors"
- note added: "E-SWITCH"
- note added: "POWER RAIL STATUS"
- note removed: "Connection to kicker board"
- note removed: "Connection to main board for motors"
- moved on the sheet: H1, H2, H3, J4, J5, J6, R1, R2

Commit message: Versão final com inclusão de test_points
Parts:
- added TP10: 5V, TestPoint:TestPoint_THTPad_D2.0mm_Drill1.0mm, symbol Connector:TestPoint
- added TP11: 3.3V, TestPoint:TestPoint_THTPad_D2.0mm_Drill1.0mm, symbol Connector:TestPoint
- added TP12: V_MON, TestPoint:TestPoint_THTPad_D2.0mm_Drill1.0mm, symbol Connector:TestPoint
- added TP13: V_BAT, TestPoint:TestPoint_THTPad_D2.0mm_Drill1.0mm, symbol Connector:TestPoint
- added TP9: 12V, TestPoint:TestPoint_THTPad_D2.0mm_Drill1.0mm, symbol Connector:TestPoint
Connections:
- net +12V: now also TP9.1
- net +3.3V: now also TP11.1
- net +5V: now also TP10.1
- net VMon: now also TP12.1
- net V_{ BATT}: now also TP13.1
Other:
- moved on the sheet: C8, D3, D5, D6, D7, H2, H3, J7, Q1, R10, R12, R5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

Commit message: DRC warnings solving
Parts:
- removed J2: XT30PW-F, Connector_AMASS:AMASS_XT30PW-F_1x02_P2.50mm_Horizontal, symbol XT30PW-F:XT30PW-F
- added J2: XT30PW-M, oxebots:AMASS_XT30PW-M, symbol oxebots:XT30PW-M
- C1, C2, C3, C9: KiLib_Generator (none) -> capacitor/THT/other
- C11: KiLib_Generator (none) -> capacitor/SMD/elec_round_polarized
- C7: renamed from C6; KiLib_Generator (none) -> capacitor/SMD/elec_round_polarized
- C8: renamed from C7; KiLib_Generator (none) -> capacitor/SMD/elec_round_polarized
- D4: renamed from D5; KiLib_Generator (none) -> SMD_2terminal_chip_molded
- D5: renamed from D6; KiLib_Generator (none) -> SMD_2terminal_chip_molded
- D6: renamed from D4; KiLib_Generator (none) -> diode/THT
- D7, R10, R13, R9: KiLib_Generator (none) -> SMD_2terminal_chip_molded
- J3: footprint Connector_AMASS:AMASS_XT30PW-M_1x02_P2.50mm_Horizontal -> oxebots:AMASS_XT30PW-M
- R11: renamed from R12; KiLib_Generator (none) -> SMD_2terminal_chip_molded
- R12: renamed from R11; KiLib_Generator (none) -> SMD_2terminal_chip_molded
- R4: renamed from R3; KiLib_Generator (none) -> SMD_2terminal_chip_molded
- R5: renamed from R4; KiLib_Generator (none) -> SMD_2terminal_chip_molded
- R7: renamed from R6; KiLib_Generator (none) -> SMD_2terminal_chip_molded
- R8: renamed from R7; KiLib_Generator (none) -> SMD_2terminal_chip_molded
- R_ADJ1, R_ADJ2, R_ADJ3: KiLib_Generator (none) -> potentiometer/SMD
- TP15: renamed from TP1; footprint TestPoint:TestPoint_Pad_D1.0mm -> Connector_Wire:SolderWirePad_1x01_SMD_5x10mm
- renumbered C8 to C4, C4 to C5, C5 to C6, D3 to D1, D1 to D2, D2 to D3, H3 to H2, H2 to H3, J7 to J4, J4 to J5, J5 to J6, J6 to J7, R5 to R1, R1 to R2, R2 to R3, R8 to R6
Connections:
- net GND: now also J2.N
- net V_{ BATT}: now also J2.P
- net Net-(J4-Pin_2): now reaches J5.2 (Pin_2), TP6.1
- net Net-(D3-K): now reaches C10.2, D8.1 (K), L3.1, U3.8 (PH)
- net Net-(D3-K): now also C4.1, D1.1 (K), Q1.1 (G), R1.1, R6.2
- net Net-(U4-BOOT): now reaches C10.1, U3.1 (BOOT)
- net Net-(J6-Pin_2): now reaches J7.2 (Pin_2), TP3.1
- net Net-(J5-Pin_2): now reaches J6.2 (Pin_2), TP8.1
- net Net-(D7-K): now reaches C5.2, D2.1 (K), L1.1, U1.8 (PH)
- net Net-(D2-K): now reaches C6.2, D3.1 (K), L2.1, U2.8 (PH)

Commit message: Board layout review and refresh fabrication outputs
Parts:
- removed J2: XT30PW-M, oxebots:AMASS_XT30PW-M, symbol oxebots:XT30PW-M
- F1: footprint Fuse:Fuseholder_Blade_Mini_Keystone_3568 -> Fuse:Fuse_Blade_Mini_directSolder
Connections:
- net Net-(D3-K) renamed Q1_GATE
- net Q1_GATE: no longer C10.2, D8.1 (K), L3.1, U3.8 (PH)
- new net SW_12V: C10.2, D8.1 (K), L3.1, U3.8 (PH)
Other:
- note removed: "Connector for Motors"
