File: pcbs/power/untitled.kicad_sch (KiCad schematic)
At the start: 33 parts, among them U1 TPS5430DDA, U2 TPS5430DDA, U4 TPS5430DDA

Commit message: Atualização para versão 10.0 do kicad Condensação do Layout Mudança no circuito V_mon para diminuir impedância de saída Implementação de Circuito "E-Switch" low side Resolução de EDR's no esquemático e PCB
Parts:
- removed C12, C7: 220uF, Capacitor_SMD:CP_Elec_6.3x7.7, symbol Device:C_US
- removed C2, C3, C8: 10uF, Capacitor_SMD:C_1206_3216Metric, symbol PCM_Capacitor_AKL:C_Generic
- removed C20: 220uF, Capacitor_SMD:CP_Elec_8x6.2, symbol Device:C_US
- removed C4, C5, C6: 0.01uF, Capacitor_SMD:C_0201_0603Metric, symbol PCM_Capacitor_AKL:C_Generic
- removed D2, D3, D7: B340, Diode_SMD:D_SMC, symbol Diode:B340
- removed D4, D5, D6: LED, LED_SMD:LED_0805_2012Metric, symbol Device:LED
- removed L1, L2, L4: 22uH, Inductor_SMD:L_6.3x6.3_H3, symbol Device:L_Iron
- removed R15, R9: 1k, PCM_Resistor_SMD_AKL:R_0805_2012Metric, symbol Device:R_US
- removed R16, R3, R6: 10k, PCM_Resistor_SMD_AKL:R_0805_2012Metric, symbol Device:R_US
- removed R4: 2.7k, PCM_Resistor_SMD_AKL:R_0805_2012Metric, symbol Device:R_US
- removed R5: 5.6k, PCM_Resistor_SMD_AKL:R_0805_2012Metric, symbol Device:R_US
- removed R7: 330, PCM_Resistor_SMD_AKL:R_0805_2012Metric, symbol Device:R_US
- removed R8: 120, PCM_Resistor_SMD_AKL:R_0805_2012Metric, symbol Device:R_US
- removed R_ADJ1, R_ADJ2: 1k, PCM_Potentiometer_SMD_AKL:Potentiometer_Bourns_3314G_Vertical, symbol Device:R_Potentiometer_Trim_US
- removed R_ADJ4: 220, PCM_Potentiometer_SMD_AKL:Potentiometer_Bourns_3314G_Vertical, symbol Device:R_Potentiometer_Trim_US
- removed U1, U2, U4: TPS5430DDA, PCM_Package_SO_AKL:Texas_HSOP-8-1EP_3.9x4.9mm_P1.27mm, symbol Regulator_Switching:TPS5430DDA
Connections:
- no-connect marks 3 -> 0
Other:
- note removed: "+12V_ALW_BUCK"
- note removed: "+3V3_ALW_BUCK"
- note removed: "+5V_ALW_BUCK"
- note removed: "POWER RAIL STATUS"
