File: pcbs/main/imu.kicad_sch (KiCad schematic)
At the start: 1 part

Commit message: fea: add jumpers to I2C encoders config
Connections:
- net IMU_SLA renamed IMU_SDA
Other:
- title: (none) -> SSL main board
Changed lines of the file:
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@@
 	(generator_version "9.0")
 	(paper "A4")
+	(title_block
+		(title "SSL main board")
+	)
 	(wire
 		(pts
@@
 		)
 	)
-	(hierarchical_label "IMU_SLA"
+	(hierarchical_label "IMU_SDA"
 		(shape bidirectional)
 		(at 121.92 92.71 180)

Commit message: wip: change radio footprint
Parts:
- renumbered IMU to IMU1
Changed lines of the file:
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@@
 		(dnp no)
 		(fields_autoplaced yes)
-		(property "Reference" "IMU"
+		(property "Reference" "IMU1"
 			(at 138.43 90.1699 0)
 			(effects
@@
 			(project ""
 				(path "/8ab8953a-1156-4e8b-85bc-154005b38a27/97614e73-f067-42e4-a0bb-405069e0b536"
-					(reference "IMU")
+					(reference "IMU1")
 					(unit 1)
 				)

Commit message: feat: association of footprints
Parts:
- IMU1: footprint (none) -> Connector_PinSocket_2.00mm:PinSocket_1x08_P2.00mm_Vertical
Changed lines of the file:
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@@
 			)
 		)
-		(property "Footprint" ""
+		(property "Footprint" "Connector_PinSocket_2.00mm:PinSocket_1x08_P2.00mm_Vertical"
 			(at 135.89 90.17 0)
 			(effects
