File: pcbs/main/esp32.kicad_sch (KiCad schematic)
At the start: 1 part, among them U1 ESP32-DEVKITC-32U

Commit message: Re-routing
Connections:
- net M1_DIR: now also U1.8 (IO33); no longer U1.28 (IO17)
- net M2_DIR: now also U1.9 (IO25); no longer U1.27 (IO16)
- net M2_PWM: now also U1.10 (IO26); no longer U1.8 (IO33)
- net M3_PWM: now also U1.12 (IO14); no longer U1.9 (IO25)
- net M4_DIR: now also U1.28 (IO17); no longer U1.12 (IO14)
- net M4_PWM: now also U1.27 (IO16); no longer U1.10 (IO26)
Changed lines of the file:
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@@
 	(wire
 		(pts
-			(xy 133.35 73.66) (xy 115.57 73.66)
+			(xy 57.15 66.04) (xy 74.93 66.04)
 		)
 		(stroke
@@
 	(wire
 		(pts
-			(xy 74.93 71.12) (xy 57.15 71.12)
+			(xy 115.57 76.2) (xy 133.35 76.2)
 		)
 		(stroke
@@
 	(wire
 		(pts
-			(xy 74.93 76.2) (xy 57.15 76.2)
+			(xy 115.57 73.66) (xy 133.35 73.66)
 		)
 		(stroke
@@
 	(wire
 		(pts
-			(xy 57.15 66.04) (xy 74.93 66.04)
+			(xy 57.15 71.12) (xy 74.93 71.12)
 		)
 		(stroke
@@
 	(wire
 		(pts
-			(xy 133.35 76.2) (xy 115.57 76.2)
+			(xy 57.15 68.58) (xy 74.93 68.58)
 		)
 		(stroke
@@
 	(wire
 		(pts
-			(xy 57.15 68.58) (xy 74.93 68.58)
+			(xy 57.15 76.2) (xy 74.93 76.2)
 		)
 		(stroke
@@
 	(hierarchical_label "M1_DIR"
 		(shape output)
-		(at 133.35 73.66 0)
-		(effects
-			(font
-				(size 1.27 1.27)
-			)
-			(justify left)
+		(at 57.15 66.04 180)
+		(effects
+			(font
+				(size 1.27 1.27)
+			)
+			(justify right)
 		)
 	)
@@
 	(hierarchical_label "M4_PWM"
 		(shape output)
-		(at 57.15 71.12 180)
-		(effects
-			(font
-				(size 1.27 1.27)
-			)
-			(justify right)
+		(at 133.35 76.2 0)
+		(effects
+			(font
+				(size 1.27 1.27)
+			)
+			(justify left)
 		)
 	)
@@
 	(hierarchical_label "M2_DIR"
 		(shape output)
-		(at 133.35 76.2 0)
-		(effects
-			(font
-				(size 1.27 1.27)
-			)
-			(justify left)
+		(at 57.15 68.58 180)
+		(effects
+			(font
+				(size 1.27 1.27)
+			)
+			(justify right)
 		)
 	)
@@
 	(hierarchical_label "M4_DIR"
 		(shape output)
-		(at 57.15 76.2 180)
-		(effects
-			(font
-				(size 1.27 1.27)
-			)
-			(justify right)
+		(at 133.35 73.66 0)
+		(effects
+			(font
+				(size 1.27 1.27)
+			)
+			(justify left)
 		)
 	)
@@
 	(hierarchical_label "M2_PWM"
 		(shape output)
-		(at 57.15 66.04 180)
+		(at 57.15 71.12 180)
 		(effects
 			(font
@@
 	(hierarchical_label "M3_PWM"
 		(shape output)
-		(at 57.15 68.58 180)
-		(effects
-			(font
+		(at 57.15 76.2 180)
+		(effects
+			(font
