File: pcbs/main/esp32.kicad_sch (KiCad schematic)
At the start: 1 part, among them U1 ESP32-DEVKITC-32U

Commit message: alteração de layout utilizado em teste para calibração dos encoders AS5600 implementando comunicação no barramento I2C
Connections:
- net MUX_A: now reaches U1.13 (IO12)
- net MUX_B: now reaches U1.23 (IO15)
- no-connect marks 9 -> 7
