File: pcbs/main/radio.kicad_sch (KiCad schematic)
At the start: 3 parts

Commit message: main
Parts:
- removed PCB1: ~, Oxebots:NRF24L01_PWR_ADP, symbol oxebots:NRF24L01_PWR_ADP
- added C14, C15, C16: 10uF, Capacitor_SMD:C_1206_3216Metric, symbol Device:C
- added U2: AMS1117-3.3, Package_TO_SOT_SMD:SOT-223-3_TabPin2, symbol Regulator_Linear:AMS1117-3.3
- C13: value 100 nF -> 10uF; footprint PCM_Capacitor_THT_AKL:C_Disc_D5.0mm_W2.5mm_P2.50mm -> Capacitor_SMD:C_1206_3216Metric
Connections:
- net +3.3V: now also C14.1, U2.3 (VI)
- net GND: now also PCB2.1 (GND_{out}), C14.2, C15.2, C16.2, U2.1 (GND)
- net RADIO_CE: now also PCB2.2 (CE)
- net RADIO_CNS: now also PCB2.6 (CSN)
- net RADIO_IRQ: now also PCB2.8 (IRQ)
- net RADIO_MISO: now also PCB2.4 (MISO)
- net RADIO_MOSI: now also PCB2.7 (MOSI)
- net RADIO_SCK: now also PCB2.3 (SCK)
- net D3.3V: now reaches PCB2.5 (VCC_{out})
- net D3.3V: now also C15.1, C16.1, U2.2 (VO)
Other:
- moved on the sheet: C13, PCB2
