File: pcbs/main/power.kicad_sch (KiCad schematic)
At the start: 5 parts, among them J2 JST_XH_B3B, J3 XT30PW-M

Commit message: Fix jumpers
Parts:
- renumbered J2 to J3, J3 to J4
Changed lines of the file:
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@@
 		(on_board yes)
 		(dnp no)
-		(property "Reference" "J2"
+		(property "Reference" "J3"
 			(at 31.75 74.9301 0)
 			(effects
@@
 			(project ""
 				(path "/8ab8953a-1156-4e8b-85bc-154005b38a27/8685a131-80f6-4b62-a6fe-8696f4df0910"
-					(reference "J2")
+					(reference "J3")
 					(unit 1)
 				)
@@
 		(dnp no)
 		(fields_autoplaced yes)
-		(property "Reference" "J3"
+		(property "Reference" "J4"
 			(at 33.02 24.13 0)
 			(effects
@@
 			(project ""
 				(path "/8ab8953a-1156-4e8b-85bc-154005b38a27/8685a131-80f6-4b62-a6fe-8696f4df0910"
-					(reference "J3")
+					(reference "J4")
 					(unit 1)
 				)

Commit message: Preliminary placing components
Connections:
- net +3.3V: no longer J3.3 (Pin_3)
- new net +5V: J3.3 (Pin_3)
Changed lines of the file:
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@@
-	)
-	(junction
-		(at 44.45 73.66)
-		(diameter 0)
-		(color 0 0 0 0)
-	)
-	(junction
-		(at 44.45 71.12)
-		(diameter 0)
-		(color 0 0 0 0)
 	)
 	(junction
@@
 	(junction
 		(at 45.72 71.12)
+		(diameter 0)
+		(color 0 0 0 0)
+	)
+	(junction
+		(at 44.45 73.66)
 		(diameter 0)
 		(color 0 0 0 0)
@@
 	(wire
 		(pts
-			(xy 44.45 73.66) (xy 44.45 71.12)
-		)
-		(stroke
-			(width 0)
-			(type default)
-		)
-	)
-	(wire
-		(pts
 			(xy 41.91 31.75) (xy 48.26 31.75)
 		)
@@
 		(pts
 			(xy 45.72 71.12) (xy 45.72 67.31)
-		)
-		(stroke
-			(width 0)
-			(type default)
-		)
-	)
-	(wire
-		(pts
-			(xy 44.45 71.12) (xy 44.45 64.77)
 		)
 		(stroke
@@
 		(pts
 			(xy 48.26 31.75) (xy 48.26 27.94)
+		)
+		(stroke
+			(width 0)
+			(type default)
+		)
+	)
+	(wire
+		(pts
+			(xy 44.45 64.77) (xy 44.45 73.66)
+		)
+		(stroke
+			(width 0)
+			(type default)
+		)
+	)
+	(wire
+		(pts
+			(xy 44.45 73.66) (xy 50.8 73.66)
 		)
 		(stroke
@@
 	(wire
 		(pts
-			(xy 39.37 71.12) (xy 44.45 71.12)
-		)
-		(stroke
-			(width 0)
-			(type default)
-		)
-	)
-	(wire
-		(pts
 			(xy 45.72 71.12) (xy 50.8 71.12)
 		)
@@
 	(wire
 		(pts
-			(xy 44.45 71.12) (xy 45.72 71.12)
+			(xy 39.37 71.12) (xy 45.72 71.12)
 		)
 		(stroke
@@
 		)
 		(stroke
-			(width 0)
-			(type default)
-		)
-	)
-	(wire
-		(pts
-			(xy 44.45 73.66) (xy 50.8 73.66)
-		)
-		(stroke
