File: pcbs/kicker/Kicker_LT3751_OxeBots.kicad_pcb (KiCad board)
At the start: 2 copper layers, 100.7 x 127.9 mm, 0 parts

Commit message: First commit of Kicker Board
Parts:
- added C1: 1000uF, Capacitor_THT:CP_Radial_D8.0mm_P5.00mm, F.Cu at (29.7, 56.5)
- added C10: 100nF, Capacitor_THT:C_Disc_D5.0mm_W2.5mm_P2.50mm, F.Cu at (85.0, 124.0)
- added C11: 100nF, Capacitor_THT:C_Disc_D5.0mm_W2.5mm_P2.50mm, F.Cu at (63.0, 134.0)
- added C12: 100nF, Capacitor_THT:C_Disc_D5.0mm_W2.5mm_P2.50mm, F.Cu at (88.5, 136.6)
- added C13: 100nF, Capacitor_THT:C_Disc_D5.0mm_W2.5mm_P2.50mm, F.Cu at (77.3, 123.8)
- added C14: 100nF, Capacitor_THT:C_Disc_D5.0mm_W2.5mm_P2.50mm, F.Cu at (93.1, 124.7)
- added C15: 220uF, Capacitor_THT:CP_Radial_D8.0mm_P5.00mm, F.Cu at (103.2, 116.7)
- added C2: 100nF, Capacitor_THT:C_Disc_D5.0mm_W2.5mm_P2.50mm, F.Cu at (65.0, 120.0)
- added C3: 10nF, Capacitor_THT:C_Rect_L19.0mm_W6.0mm_P15.00mm_MKS4, F.Cu at (135.1, 106.6)
- added C4: 100uF, Capacitor_THT:CP_Radial_D30.0mm_P10.00mm_SnapIn, F.Cu at (136.1, 48.3)
- added C5: 100uF, Capacitor_THT:CP_Radial_D30.0mm_P10.00mm_SnapIn, F.Cu at (136.1, 162.3)
- added C6: 22nF, Capacitor_THT:C_Rect_L7.0mm_W4.5mm_P5.00mm, F.Cu at (87.4, 82.5)
- added C7: 100nF, Capacitor_THT:C_Disc_D5.0mm_W2.5mm_P2.50mm, F.Cu at (80.0, 117.0)
- added C8: 100nF, Capacitor_THT:C_Disc_D5.0mm_W2.5mm_P2.50mm, F.Cu at (81.0, 112.0)
- added C9: 10nF, Capacitor_THT:C_Disc_D5.0mm_W2.5mm_P2.50mm, F.Cu at (115.0, 106.0)
- added D1: MUR460, Diode_THT:D_DO-201AD_P12.70mm_Horizontal, F.Cu at (136.0, 69.8)
- added D2: MUR460, Diode_THT:D_DO-201AD_P12.70mm_Horizontal, F.Cu at (136.0, 139.6)
- added D3: LED, LED_THT:LED_D3.0mm_Clear, F.Cu at (48.1, 138.1)
- added D4: LED, LED_THT:LED_D3.0mm_Clear, F.Cu at (53.2, 146.5)
- added IC1: LT3751, Package_SO:TSSOP-20-1EP_4.4x6.5mm_P0.65mm_EP2.15x3.35mm, F.Cu at (81.6, 106.1)
- added J1: XT30PW-F, oxebots_connectors:AMASS_XT30PW-F, F.Cu at (72.2, 63.7)
- added J2: XT30PW-F, oxebots_connectors:AMASS_XT30PW-F, F.Cu at (49.9, 117.5)
- added J3: ~, Connector_PinHeader_2.54mm:PinHeader_1x06_P2.54mm_Vertical, F.Cu at (72.5, 145.2)
- added J4: SOL, TerminalBlock_Phoenix:TerminalBlock_Phoenix_MKDS-1,5-2_1x02_P5.00mm_Horizontal, F.Cu at (117.6, 150.7)
- added PS1: B1215S, Converter_DCDC:Converter_DCDC_Murata_MEE1SxxxxSC_THT, F.Cu at (89.8, 119.5)
- added Q1: IRFB4227, Package_TO_SOT_THT:TO-220-3_Vertical, F.Cu at (71.9, 83.5)
- added Q2: FGH60N60SMD, Package_TO_SOT_THT:TO-247-3_Vertical, F.Cu at (115.3, 129.3)
- added Q3: BC547, Package_TO_SOT_THT:TO-92_Inline, F.Cu at (70.5, 127.9)
- added Q4: BC547, Package_TO_SOT_THT:TO-92_Inline, F.Cu at (70.5, 133.7)
- added R1: 4,7K, Resistor_THT:R_Axial_DIN0922_L20.0mm_D9.0mm_P7.62mm_Vertical, F.Cu at (87.4, 70.7)
- added R10: ?, Resistor_THT:R_Axial_DIN0207_L6.3mm_D2.5mm_P7.62mm_Horizontal, F.Cu at (123.0, 81.0)
- added R11: ?, Resistor_THT:R_Axial_DIN0207_L6.3mm_D2.5mm_P7.62mm_Horizontal, F.Cu at (123.0, 76.0)
- added R12: 1M, Resistor_THT:R_Axial_DIN0207_L6.3mm_D2.5mm_P7.62mm_Horizontal, F.Cu at (139.0, 105.0)
- added R13: 220R, Resistor_THT:R_Axial_DIN0207_L6.3mm_D2.5mm_P7.62mm_Horizontal, F.Cu at (84.4, 140.4)
- added R14: R, Resistor_THT:R_Axial_DIN0207_L6.3mm_D2.5mm_P7.62mm_Horizontal, F.Cu at (101.7, 128.2)
- added R15: R, Resistor_THT:R_Axial_DIN0207_L6.3mm_D2.5mm_P7.62mm_Horizontal, F.Cu at (109.3, 132.0)
- added R16: R, Resistor_THT:R_Axial_DIN0207_L6.3mm_D2.5mm_P7.62mm_Horizontal, F.Cu at (123.0, 115.0)
- added R17: R, Resistor_THT:R_Axial_DIN0207_L6.3mm_D2.5mm_P7.62mm_Horizontal, F.Cu at (138.9, 100.4)
- added R18: 1K, Resistor_THT:R_Axial_DIN0207_L6.3mm_D2.5mm_P7.62mm_Horizontal, F.Cu at (54.0, 152.0)
- added R19: 1K, Resistor_THT:R_Axial_DIN0207_L6.3mm_D2.5mm_P7.62mm_Horizontal, F.Cu at (41.0, 131.0)
- added R2: 39K, Resistor_THT:R_Axial_DIN0207_L6.3mm_D2.5mm_P7.62mm_Horizontal, F.Cu at (93.0, 100.1)
- added R20: 10K, Resistor_THT:R_Axial_DIN0207_L6.3mm_D2.5mm_P7.62mm_Horizontal, F.Cu at (62.0, 139.0)
- added R21: 10K, Resistor_THT:R_Axial_DIN0207_L6.3mm_D2.5mm_P7.62mm_Horizontal, F.Cu at (88.0, 132.0)
- added R22: 10K, Resistor_THT:R_Axial_DIN0207_L6.3mm_D2.5mm_P7.62mm_Horizontal, F.Cu at (73.0, 139.0)
- added R23: 10K, Resistor_THT:R_Axial_DIN0207_L6.3mm_D2.5mm_P7.62mm_Horizontal, F.Cu at (67.0, 112.0)
- added R3: 18K, Resistor_THT:R_Axial_DIN0207_L6.3mm_D2.5mm_P7.62mm_Horizontal, F.Cu at (67.3, 99.3)
- added R4: 39K, Resistor_THT:R_Axial_DIN0207_L6.3mm_D2.5mm_P7.62mm_Horizontal, F.Cu at (71.6, 99.3)
- added R5: 10R, Resistor_THT:R_Axial_DIN0207_L6.3mm_D2.5mm_P7.62mm_Horizontal, F.Cu at (80.2, 99.2)
- added R6: 25m (NOTA 1), Resistor_SMD:R_2512_6332Metric, F.Cu at (63.7, 77.3)
- added R7: 220R, Resistor_THT:R_Axial_DIN0207_L6.3mm_D2.5mm_P7.62mm_Horizontal, F.Cu at (77.0, 135.0)
- added R8: 1,5K, Resistor_THT:R_Axial_DIN0207_L6.3mm_D2.5mm_P7.62mm_Horizontal, F.Cu at (75.9, 99.3)
- added R9: ?, Resistor_THT:R_Axial_DIN0207_L6.3mm_D2.5mm_P7.62mm_Horizontal, F.Cu at (123.0, 86.0)
- added SW1: SW_Push, Button_Switch_THT:SW_PUSH_6mm_H7.3mm, F.Cu at (198.6, 84.2)
- added T1: DCT15EFD-U44S003, oxebots_transformer:TRANS_U44S003_TDK, F.Cu at (110.4, 78.2)
- added U1: LM7805_TO220, Package_TO_SOT_THT:TO-220-3_Vertical, F.Cu at (55.0, 136.0)
- added U2: HCPL-3120, Package_DIP:DIP-8_W7.62mm, F.Cu at (94.1, 137.1)
Routing:
- added copper zone on F.Cu, net VCAP
Other:
- board size 100.7 x 127.9 mm -> 117.9 x 140 mm

Commit message: Updated feedback circuit
Parts:
- removed IC1: LT3751, Package_SO:TSSOP-20-1EP_4.4x6.5mm_P0.65mm_EP2.15x3.35mm
- added C16: 100nF, Capacitor_THT:C_Disc_D5.0mm_W2.5mm_P2.50mm, F.Cu at (229.4, 123.1)
- added C17: 100nF, Capacitor_THT:C_Disc_D5.0mm_W2.5mm_P2.50mm, F.Cu at (236.0, 111.0)
- added C18: 100nF, Capacitor_THT:C_Disc_D5.0mm_W2.5mm_P2.50mm, F.Cu at (236.0, 115.0)
- added C19: 100nF, Capacitor_THT:C_Disc_D5.0mm_W2.5mm_P2.50mm, F.Cu at (236.0, 119.1)
- added C20: C, Capacitor_THT:C_Disc_D5.0mm_W2.5mm_P2.50mm, F.Cu at (236.0, 123.1)
- added C21: 100nF, Capacitor_THT:C_Rect_L19.0mm_W6.0mm_P15.00mm_MKS4, F.Cu at (261.8, 102.1)
- added C22: 100nF, Capacitor_THT:C_Rect_L19.0mm_W6.0mm_P15.00mm_MKS4, F.Cu at (261.8, 109.7)
- added D5: 1N4712A, Diode_THT:D_DO-41_SOD81_P10.16mm_Horizontal, F.Cu at (185.6, 98.5)
- added D6: D_Zener, Diode_THT:D_DO-35_SOD27_P7.62mm_Horizontal, F.Cu at (270.7, 58.5)
- added F1: 10A, Fuse:Fuse_Blade_ATO_directSolder, F.Cu at (265.2, 117.2)
- added J5: Conn_01x04, Connector_PinHeader_2.54mm:PinHeader_1x04_P2.54mm_Vertical, F.Cu at (201.4, 102.9)
- added J6: XT30PW-F, oxebots_connectors:AMASS_XT30PW-M, F.Cu at (129.3, 134.9)
- added J7: Conn_01x05, Connector_PinHeader_2.54mm:PinHeader_1x05_P2.54mm_Vertical, F.Cu at (48.9, 129.4)
- added J8: Conn_01x08, Connector_PinHeader_2.54mm:PinHeader_1x08_P2.54mm_Vertical, F.Cu at (53.5, 121.9)
- added JP1: ~, Jumper:SolderJumper-3_P1.3mm_Open_Pad1.0x1.5mm, F.Cu at (186.6, 128.9)
- added Q5: BC547, Package_TO_SOT_THT:TO-92_Inline, F.Cu at (207.3, 116.1)
- added Q6: BC547, Package_TO_SOT_THT:TO-92_Inline, F.Cu at (207.3, 121.9)
- added R24: 470R, Resistor_THT:R_Axial_DIN0207_L6.3mm_D2.5mm_P7.62mm_Horizontal, F.Cu at (239.4, 56.4)
- added R25: 27k, Resistor_THT:R_Axial_DIN0207_L6.3mm_D2.5mm_P7.62mm_Horizontal, F.Cu at (239.4, 60.4)
- added R26: 1k, Resistor_THT:R_Axial_DIN0207_L6.3mm_D2.5mm_P7.62mm_Horizontal, F.Cu at (239.4, 64.5)
- added R27: 10k, Resistor_THT:R_Axial_DIN0207_L6.3mm_D2.5mm_P7.62mm_Horizontal, F.Cu at (239.4, 68.5)
- added R28: 18k, Resistor_THT:R_Axial_DIN0207_L6.3mm_D2.5mm_P7.62mm_Horizontal, F.Cu at (239.4, 72.6)
- added R29: 100k, Resistor_THT:R_Axial_DIN0207_L6.3mm_D2.5mm_P7.62mm_Horizontal, F.Cu at (239.4, 76.6)
- added R30: 330k, Resistor_THT:R_Axial_DIN0207_L6.3mm_D2.5mm_P7.62mm_Horizontal, F.Cu at (239.4, 80.7)
- added R31: 4.7k, Resistor_THT:R_Axial_DIN0207_L6.3mm_D2.5mm_P7.62mm_Horizontal, F.Cu at (239.4, 84.7)
- added R32: 4.7k, Resistor_THT:R_Axial_DIN0207_L6.3mm_D2.5mm_P7.62mm_Horizontal, F.Cu at (239.4, 88.8)
- added R33: 330k, Resistor_THT:R_Axial_DIN0207_L6.3mm_D2.5mm_P7.62mm_Horizontal, F.Cu at (250.2, 52.3)
- added R34: 330k, Resistor_THT:R_Axial_DIN0207_L6.3mm_D2.5mm_P7.62mm_Horizontal, F.Cu at (250.2, 56.4)
- added R35: 27k, Resistor_THT:R_Axial_DIN0207_L6.3mm_D2.5mm_P7.62mm_Horizontal, F.Cu at (250.2, 60.4)
- added R36: 47k, Resistor_THT:R_Axial_DIN0207_L6.3mm_D2.5mm_P7.62mm_Horizontal, F.Cu at (250.2, 64.5)
- added R37: 470R, Resistor_THT:R_Axial_DIN0207_L6.3mm_D2.5mm_P7.62mm_Horizontal, F.Cu at (250.2, 68.5)
- added R38: R, Resistor_THT:R_Axial_DIN0207_L6.3mm_D2.5mm_P7.62mm_Horizontal, F.Cu at (250.2, 72.6)
- added R39: 100K, Resistor_THT:R_Axial_DIN0207_L6.3mm_D2.5mm_P7.62mm_Horizontal, F.Cu at (250.2, 76.6)
- added R40: R, Resistor_THT:R_Axial_DIN0207_L6.3mm_D2.5mm_P7.62mm_Horizontal, F.Cu at (250.2, 80.7)
- added R41: 4.7k, Resistor_THT:R_Axial_DIN0207_L6.3mm_D2.5mm_P7.62mm_Horizontal, F.Cu at (250.2, 84.7)
- added R42: 4.7k, Resistor_THT:R_Axial_DIN0207_L6.3mm_D2.5mm_P7.62mm_Horizontal, F.Cu at (250.2, 88.8)
- added RV1: 100k, Potentiometer_THT:Potentiometer_Bourns_3296W_Vertical, F.Cu at (277.2, 53.5)
- added U3: STM32F030F4Px, Package_SO:TSSOP-20_4.4x6.5mm_P0.65mm, F.Cu at (210.1, 128.5)
- added U4: PC817, Package_DIP:DIP-4_W7.62mm, F.Cu at (185.4, 109.3)
- added U7: LM358, Package_DIP:DIP-8_W7.62mm, F.Cu at (196.1, 114.9)
- added U8: HCNR201, Package_DIP:DIP-8_W7.62mm_LongPads, F.Cu at (247.9, 117.5)
- C1: value 1000uF -> 100nF; footprint Capacitor_THT:CP_Radial_D8.0mm_P5.00mm -> Capacitor_THT:C_Disc_D5.0mm_W2.5mm_P2.50mm
- C10: value 100nF -> 10nF
- C11, C8: value 100nF -> 220uF; footprint Capacitor_THT:C_Disc_D5.0mm_W2.5mm_P2.50mm -> Capacitor_THT:CP_Radial_D8.0mm_P5.00mm
- C2: value 100nF -> 1000uF; footprint Capacitor_THT:C_Disc_D5.0mm_W2.5mm_P2.50mm -> Capacitor_THT:CP_Radial_D8.0mm_P5.00mm
- C3: value 10nF -> 100nF; footprint Capacitor_THT:C_Rect_L19.0mm_W6.0mm_P15.00mm_MKS4 -> Capacitor_THT:C_Disc_D5.0mm_W2.5mm_P2.50mm
- C4: value 100uF -> 100nF; footprint Capacitor_THT:CP_Radial_D30.0mm_P10.00mm_SnapIn -> Capacitor_THT:C_Rect_L19.0mm_W6.0mm_P15.00mm_MKS4
- C5: value 100uF -> 820uF
- C6: value 22nF -> 820uF; footprint Capacitor_THT:C_Rect_L7.0mm_W4.5mm_P5.00mm -> Capacitor_THT:CP_Radial_D30.0mm_P10.00mm_SnapIn
- C7: value 100nF -> 22nF; footprint Capacitor_THT:C_Disc_D5.0mm_W2.5mm_P2.50mm -> Capacitor_THT:C_Rect_L7.0mm_W4.5mm_P5.00mm
- C9: value 10nF -> 100nF
- D1: value MUR460 -> SMBJ26A; footprint Diode_THT:D_DO-201AD_P12.70mm_Horizontal -> Diode_SMD:D_SMB_Handsoldering
- D3, D4: value LED -> 1.5KE300A; footprint LED_THT:LED_D3.0mm_Clear -> Diode_THT:D_DO-201AE_P15.24mm_Horizontal
- J1: footprint oxebots_connectors:AMASS_XT30PW-F -> oxebots_connectors:AMASS_XT30PW-M
- J2: value XT30PW-F -> CONN_BUCK; footprint oxebots_connectors:AMASS_XT30PW-F -> Connector_PinSocket_2.54mm:PinSocket_1x04_P2.54mm_Vertical
- J3: value ~ -> Conn_01x02; footprint Connector_PinHeader_2.54mm:PinHeader_1x06_P2.54mm_Vertical -> Connector_JST:JST_XH_B2B-XH-A_1x02_P2.50mm_Vertical
- J4: value SOL -> XT30PW-F; footprint TerminalBlock_Phoenix:TerminalBlock_Phoenix_MKDS-1,5-2_1x02_P5.00mm_Horizontal -> oxebots_connectors:AMASS_XT30PW-M
- Q2: value FGH60N60SMD -> CS20N60; footprint Package_TO_SOT_THT:TO-247-3_Vertical -> Package_TO_SOT_SMD:TO-263-2
- Q3: value BC547 -> CS20N60; footprint Package_TO_SOT_THT:TO-92_Inline -> Package_TO_SOT_SMD:TO-263-2
- Q4: value BC547 -> TIC106; footprint Package_TO_SOT_THT:TO-92_Inline -> Package_TO_SOT_THT:TO-220-3_Vertical
- R10: value ? -> 180k
- R11: value ? -> 510k
- R12: value 1M -> 270k
- R13: value 220R -> 3.3k
- R14, R15, R16: value R -> 220R
- R17: value R -> 3.3k
- R18: value 1K -> 3.3k
- R19: value 1K -> 220R
- R2: value 39K -> 18K
- R20, R21: value 10K -> 220R
- R22: value 10K -> 3.3k
- R23: value 10K -> 10k
- R3: value 18K -> 39K
- R9: value ? -> 300k
- SW1: footprint Button_Switch_THT:SW_PUSH_6mm_H7.3mm -> Button_Switch_THT:SW_PUSH_6mm_H4.3mm
- U1: value LM7805_TO220 -> LT3751; footprint Package_TO_SOT_THT:TO-220-3_Vertical -> Package_SO:TSSOP-20-1EP_4.4x6.5mm_P0.65mm_EP2.15x3.35mm
- U2: value HCPL-3120 -> PC817; footprint Package_DIP:DIP-8_W7.62mm -> Package_DIP:DIP-4_W7.62mm
- moved D3 237.5 mm to (262.9, 36.7), turned to 0 degrees
- moved D4 233.6 mm to (262.9, 43.5), turned to 0 degrees
- moved J3 211.2 mm to (272.6, 77.7), turned to 0 degrees
- moved C11 207.6 mm to (261.8, 74.2)
- moved C2 207.3 mm to (261.8, 55.1), turned to 0 degrees
- moved C1 200.7 mm to (222.9, 111.0), turned to 0 degrees
- moved R19 195.3 mm to (228.6, 76.6)
- moved R18 191.8 mm to (228.6, 72.6)
- moved C8 186.9 mm to (261.8, 64.6)
- moved R1 185.5 mm to (264.3, 126.3), turned to 0 degrees
- moved R23 182.4 mm to (239.4, 52.3)
- moved R20 176.5 mm to (228.6, 80.7)
- moved R13 169.0 mm to (228.6, 52.3), turned to 0 degrees
- moved R22 163.5 mm to (228.6, 88.8)
- moved C15 162.0 mm to (261.8, 83.7)
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Connections:
- C1 pad 1: UVLO_1 -> +12V
- C1 pad 2: OVLO_1 -> GND
- C10 pad 1: UVLO_2 -> LT3751_FB
- C10 pad 2: OVLO_1 -> GND
- C11 pad 1: +5V -> +3.3V
- C11 pad 2: OVLO_1 -> GND
- C12 pad 1: Net-(U2-A) -> +3.3V
- C12 pad 2: OVLO_1 -> GND
- C13 pad 1: UVLO_2 -> +12V
- C13 pad 2: OVLO_1 -> GND
- C14 pad 2: OVLO_1 -> GNDPWR
- C15 pad 2: OVLO_1 -> GNDPWR
- C2 pad 1: UVLO_1 -> +24V
- C2 pad 2: OVLO_1 -> GND
- C3 pad 1: VCAP -> +24V
- C3 pad 2: OVLO_1 -> GND
- C4 pad 2: OVLO_1 -> GNDPWR
- C5 pad 2: OVLO_1 -> GNDPWR
- C6 pad 1: Net-(C6-Pad1) -> VCAP
- C6 pad 2: Net-(Q1-D) -> GNDPWR
- C7 pad 1: UVLO_2 -> Net-(C7-Pad1)
- C7 pad 2: OVLO_1 -> Net-(Q1-D)
- C8 pad 1: UVLO_2 -> +12V
- C8 pad 2: OVLO_1 -> GND
- C9 pad 1: FB -> +12V
- C9 pad 2: OVLO_1 -> GND
- D1 pad 1: VCAP -> GND
- D1 pad 2: Net-(D1-A) -> +24V
- D3 pad 1: Net-(D3-K) -> VCAP
- D3 pad 2: Net-(D3-A) -> Net-(D3-A2)
- D4 pad 1: Net-(D4-K) -> VCAP
- D4 pad 2: Net-(D4-A) -> Net-(D4-A2)
- J1 pad N: OVLO_1 -> GND
- J1 pad P: UVLO_1 -> Net-(F1-Pad1)
- J3 pad 1: MCU_IN_ENABLE -> +3.3V
- J3 pad 2: MCU_IN_KICK -> GND
- PS1 pad 1: OVLO_1 -> GND
- PS1 pad 2: UVLO_2 -> +12V
- PS1 pad 3: OVLO_1 -> GNDPWR
- Q1 pad 3: Net-(IC1-CSP) -> Net-(Q1-S)
- Q2 pad 2: Net-(D2-A) -> Net-(D3-A2)
- Q2 pad 3: OVLO_1 -> GNDPWR
- Q3 pad 1: Net-(D3-K) -> Net-(Q3-G)
- Q3 pad 2: DONE -> Net-(D4-A2)
- Q3 pad 3: OVLO_1 -> GNDPWR
- Q4 pad 1: Net-(D4-K) -> GNDPWR
- Q4 pad 2: FAULT -> Net-(Q4-A)
- Q4 pad 3: OVLO_1 -> Net-(Q4-G)
- R1 pad 1: UVLO_1 -> +24V
- R1 pad 2: Net-(C6-Pad1) -> Net-(C7-Pad1)
- R10 pad 1: VCAP -> +12V
- R10 pad 2: Net-(R10-Pad2) -> UVLO_2
- R11 pad 1: VCAP -> +24V
- R11 pad 2: Net-(R10-Pad2) -> OVLO_1
- R12 pad 1: VCAP -> +12V
- R12 pad 2: OVLO_1 -> OVLO_2
- R13 pad 1: MCU_IN_KICK -> +15V_SEC
- R13 pad 2: Net-(U2-A) -> Net-(R13-Pad2)
- R14 pad 1: Net-(R14-Pad1) -> EXT_IN_LT3751_KICK_1
- R14 pad 2: Net-(Q2-G) -> Net-(C16-Pad1)
- R15 pad 1: Net-(Q2-G) -> MCU_OUT_KICK_1
- R15 pad 2: OVLO_1 -> Net-(C16-Pad1)
- R16 pad 1: VCAP -> Net-(R13-Pad2)
- R16 pad 2: FB -> Net-(Q2-G)
- R17 pad 1: FB -> Net-(Q2-G)
- R17 pad 2: OVLO_1 -> GNDPWR
- R18 pad 1: +5V -> +15V_SEC
- R18 pad 2: Net-(D3-A) -> Net-(R18-Pad2)
- R19 pad 1: +5V -> EXT_IN_LT3751_KICK_1
- R19 pad 2: Net-(D4-A) -> Net-(C17-Pad1)
- R2 pad 1: UVLO_1 -> Net-(U1-RDCM)
- R2 pad 2: Net-(IC1-RVTRANS) -> Net-(Q1-D)
- R20 pad 1: +5V -> MCU_OUT_KICK_2
- R20 pad 2: DONE -> Net-(C17-Pad1)
- R21 pad 1: Net-(D3-K) -> Net-(R18-Pad2)
- R21 pad 2: MCU_OUT_DONE -> Net-(Q3-G)
- R22 pad 1: +5V -> Net-(Q3-G)
- R22 pad 2: FAULT -> GNDPWR
- R23 pad 1: Net-(D4-K) -> +3.3V
- R23 pad 2: MCU_OUT_FAULT -> MCU_RST
- R3 pad 1: Net-(IC1-RDCM) -> Net-(U1-RVOUT)
- R4 pad 1: Net-(IC1-RVOUT) -> +24V
- R4 pad 2: Net-(Q1-D) -> Net-(U1-RVTRANS)
- R5 pad 1: Net-(IC1-HVGATE) -> Net-(U1-HVGATE)
- R6 pad 1: Net-(IC1-CSP) -> Net-(Q1-S)
- R6 pad 2: OVLO_1 -> GND
- R7 pad 1: MCU_IN_ENABLE -> MCU_OUT_ENABLE
- R7 pad 2: Net-(IC1-CHARGE) -> Net-(U1-CHARGE)
- R8 pad 1: Net-(IC1-RBG) -> Net-(U1-RBG)
- R8 pad 2: OVLO_1 -> GND
- R9 pad 1: VCAP -> +24V
- R9 pad 2: Net-(R10-Pad2) -> UVLO_1
- SW1 pad 1: OVLO_1 -> GND
- SW1 pad 2: Net-(R10-Pad2) -> MCU_RST
- T1 pad 1: Net-(D1-A) -> Net-(D2-A)
- T1 pad 10: OVLO_1 -> GNDPWR
- T1 pad 4: UVLO_1 -> +24V
- T1 pad 5: UVLO_1 -> +24V
- U1 pad 1: UVLO_2 -> Net-(U1-RVTRANS)
- U1 pad 2: OVLO_1 -> LT3751_UVLO_1
- U1 pad 3: +5V -> LT3751_OVLO_1
- U2 pad 1: unconnected-(U2-NC-Pad1) -> Net-(C16-Pad1)
- U2 pad 2: Net-(U2-A) -> GND
- U2 pad 3: OVLO_1 -> GNDPWR
- U2 pad 4: unconnected-(U2-NC-Pad4) -> Net-(R13-Pad2)
Routing:
- removed copper zone on F.Cu, net VCAP
Other:
- outline, holes or cut-outs redrawn

Commit message: update
Placa parcialmente desenhada, componentes posicionados
Parts:
- removed C20: C, Capacitor_THT:C_Disc_D5.0mm_W2.5mm_P2.50mm
- removed C21, C22: 100nF, Capacitor_THT:C_Rect_L19.0mm_W6.0mm_P15.00mm_MKS4
- removed D5: 1N4712A, Diode_THT:D_DO-41_SOD81_P10.16mm_Horizontal
- removed D6: D_Zener, Diode_THT:D_DO-35_SOD27_P7.62mm_Horizontal
- removed J6: XT30PW-F, oxebots_connectors:AMASS_XT30PW-M
- removed J7: Conn_01x05, Connector_PinHeader_2.54mm:PinHeader_1x05_P2.54mm_Vertical
- removed J8: Conn_01x08, Connector_PinHeader_2.54mm:PinHeader_1x08_P2.54mm_Vertical
- removed JP1: ~, Jumper:SolderJumper-3_P1.3mm_Open_Pad1.0x1.5mm
- removed Q6: BC547, Package_TO_SOT_THT:TO-92_Inline
- removed SW1: SW_Push, Button_Switch_THT:SW_PUSH_6mm_H4.3mm
- added R43: 510k, Resistor_THT:R_Axial_DIN0207_L6.3mm_D2.5mm_P7.62mm_Horizontal, F.Cu at (123.2, 54.6)
- added R44: 47k, Resistor_THT:R_Axial_DIN0207_L6.3mm_D2.5mm_P7.62mm_Horizontal, F.Cu at (118.6, 54.6)
- added R45: 33k, Resistor_THT:R_Axial_DIN0207_L6.3mm_D2.5mm_P7.62mm_Horizontal, F.Cu at (114.0, 54.6)
- added RV2: 100k, Potentiometer_THT:Potentiometer_Bourns_3296W_Vertical, F.Cu at (58.4, 88.1)
- added U5: AQV454, Package_DIP:DIP-6_W7.62mm_LongPads, F.Cu at (94.0, 138.6)
- added U6: HCNR201, Package_DIP:DIP-8_W10.16mm_LongPads, F.Cu at (104.9, 69.1)
- C1: value 100nF -> 1000uF; footprint Capacitor_THT:C_Disc_D5.0mm_W2.5mm_P2.50mm -> Capacitor_THT:CP_Radial_D8.0mm_P5.00mm
- C10: value 10nF -> 100nF
- C11: value 220uF -> 22nF; footprint Capacitor_THT:CP_Radial_D8.0mm_P5.00mm -> Capacitor_THT:C_Rect_L7.0mm_W4.5mm_P5.00mm
- C12: footprint Capacitor_THT:C_Disc_D5.0mm_W2.5mm_P2.50mm -> Capacitor_THT:C_Rect_L19.0mm_W6.0mm_P15.00mm_MKS4
- C13, C19, C3: footprint Capacitor_THT:C_Disc_D5.0mm_W2.5mm_P2.50mm -> Capacitor_SMD:C_0805_2012Metric_Pad1.18x1.45mm_HandSolder
- C15: value 220uF -> 100nF; footprint Capacitor_THT:CP_Radial_D8.0mm_P5.00mm -> Capacitor_THT:C_Disc_D5.0mm_W2.5mm_P2.50mm
- C16, C18: value 100nF -> 820uF; footprint Capacitor_THT:C_Disc_D5.0mm_W2.5mm_P2.50mm -> Capacitor_THT:CP_Radial_D30.0mm_P10.00mm_SnapIn; moved to B.Cu
- C17: value 100nF -> 220uF; footprint Capacitor_THT:C_Disc_D5.0mm_W2.5mm_P2.50mm -> Capacitor_THT:CP_Radial_D8.0mm_P5.00mm
- C2: value 1000uF -> 100nF; footprint Capacitor_THT:CP_Radial_D8.0mm_P5.00mm -> Capacitor_SMD:C_0805_2012Metric_Pad1.18x1.45mm_HandSolder
- C4: footprint Capacitor_THT:C_Rect_L19.0mm_W6.0mm_P15.00mm_MKS4 -> Capacitor_THT:C_Disc_D5.0mm_W2.5mm_P2.50mm
- C5, C6: value 820uF -> 100nF; footprint Capacitor_THT:CP_Radial_D30.0mm_P10.00mm_SnapIn -> Capacitor_SMD:C_0805_2012Metric_Pad1.18x1.45mm_HandSolder
- C7: value 22nF -> 100nF; footprint Capacitor_THT:C_Rect_L7.0mm_W4.5mm_P5.00mm -> Capacitor_SMD:C_0805_2012Metric_Pad1.18x1.45mm_HandSolder
- C8: value 220uF -> 10nF; footprint Capacitor_THT:CP_Radial_D8.0mm_P5.00mm -> Capacitor_THT:C_Disc_D5.0mm_W2.5mm_P2.50mm
- C9: value 100nF -> 1nF; footprint Capacitor_THT:C_Disc_D5.0mm_W2.5mm_P2.50mm -> Capacitor_SMD:C_0805_2012Metric_Pad1.18x1.45mm_HandSolder
- D1: value SMBJ26A -> MUR460; footprint Diode_SMD:D_SMB_Handsoldering -> Diode_THT:D_DO-201AD_P12.70mm_Horizontal
- D2: value MUR460 -> 1N4712A; footprint Diode_THT:D_DO-201AD_P12.70mm_Horizontal -> Diode_THT:D_DO-41_SOD81_P7.62mm_Horizontal
- D3: value 1.5KE300A -> 1.5KE220A
- D4: value 1.5KE300A -> SMBJ26A; footprint Diode_THT:D_DO-201AE_P15.24mm_Horizontal -> Diode_SMD:D_SMB
- F1: value 10A -> Fuse
- J2: value CONN_BUCK -> Conn_01x02; footprint Connector_PinSocket_2.54mm:PinSocket_1x04_P2.54mm_Vertical -> Connector_JST:JST_XH_B2B-XH-A_1x02_P2.50mm_Vertical
- J4: value XT30PW-F -> Conn_01x08; footprint oxebots_connectors:AMASS_XT30PW-M -> Connector_PinHeader_2.54mm:PinHeader_1x08_P2.54mm_Vertical
- J5: value Conn_01x04 -> XT30PW-F; footprint Connector_PinHeader_2.54mm:PinHeader_1x04_P2.54mm_Vertical -> oxebots_connectors:AMASS_XT30PW-M
- Q1: value IRFB4227 -> BC847; footprint Package_TO_SOT_THT:TO-220-3_Vertical -> Package_TO_SOT_SMD:SOT-23; moved to B.Cu
- Q2: value CS20N60 -> BC847; footprint Package_TO_SOT_SMD:TO-263-2 -> Package_TO_SOT_SMD:SOT-23; moved to B.Cu
- Q3: value CS20N60 -> IRFB4227; footprint Package_TO_SOT_SMD:TO-263-2 -> Package_TO_SOT_THT:TO-220-3_Vertical
- Q5: value BC547 -> FQPF20N60; footprint Package_TO_SOT_THT:TO-92_Inline -> Package_TO_SOT_THT:TO-220F-3_Vertical
- R1: value 4,7K -> 300k; footprint Resistor_THT:R_Axial_DIN0922_L20.0mm_D9.0mm_P7.62mm_Vertical -> Resistor_SMD:R_0805_2012Metric_Pad1.20x1.40mm_HandSolder
- R10: value 180k -> 1.2k; footprint Resistor_THT:R_Axial_DIN0207_L6.3mm_D2.5mm_P7.62mm_Horizontal -> Resistor_SMD:R_0805_2012Metric_Pad1.20x1.40mm_HandSolder
- R11: value 510k -> 9.1k; footprint Resistor_THT:R_Axial_DIN0207_L6.3mm_D2.5mm_P7.62mm_Horizontal -> Resistor_SMD:R_0805_2012Metric_Pad1.20x1.40mm_HandSolder
- R12: value 270k -> 10k; footprint Resistor_THT:R_Axial_DIN0207_L6.3mm_D2.5mm_P7.62mm_Horizontal -> Resistor_SMD:R_0805_2012Metric_Pad1.20x1.40mm_HandSolder
- R13: value 3.3k -> 10k; footprint Resistor_THT:R_Axial_DIN0207_L6.3mm_D2.5mm_P7.62mm_Horizontal -> Resistor_SMD:R_0805_2012Metric_Pad1.20x1.40mm_HandSolder
- R14: value 220R -> 1k; footprint Resistor_THT:R_Axial_DIN0207_L6.3mm_D2.5mm_P7.62mm_Horizontal -> Resistor_SMD:R_0805_2012Metric_Pad1.20x1.40mm_HandSolder
- R15: value 220R -> 1,5K; footprint Resistor_THT:R_Axial_DIN0207_L6.3mm_D2.5mm_P7.62mm_Horizontal -> Resistor_SMD:R_0805_2012Metric_Pad1.20x1.40mm_HandSolder
- R16, R21: value 220R -> 4.7k; footprint Resistor_THT:R_Axial_DIN0207_L6.3mm_D2.5mm_P7.62mm_Horizontal -> Resistor_SMD:R_0805_2012Metric_Pad1.20x1.40mm_HandSolder; moved to B.Cu
- R17, R22: value 3.3k -> 4.7k; footprint Resistor_THT:R_Axial_DIN0207_L6.3mm_D2.5mm_P7.62mm_Horizontal -> Resistor_SMD:R_0805_2012Metric_Pad1.20x1.40mm_HandSolder; moved to B.Cu
- R18: value 3.3k -> 18K; footprint Resistor_THT:R_Axial_DIN0207_L6.3mm_D2.5mm_P7.62mm_Horizontal -> Resistor_SMD:R_0805_2012Metric_Pad1.20x1.40mm_HandSolder
- R19: value 220R -> 39K; footprint Resistor_THT:R_Axial_DIN0207_L6.3mm_D2.5mm_P7.62mm_Horizontal -> Resistor_SMD:R_0805_2012Metric_Pad1.20x1.40mm_HandSolder
- R2: value 18K -> 510k; footprint Resistor_THT:R_Axial_DIN0207_L6.3mm_D2.5mm_P7.62mm_Horizontal -> Resistor_SMD:R_0805_2012Metric_Pad1.20x1.40mm_HandSolder
- R20: value 220R -> 10R; footprint Resistor_THT:R_Axial_DIN0207_L6.3mm_D2.5mm_P7.62mm_Horizontal -> Resistor_SMD:R_0805_2012Metric_Pad1.20x1.40mm_HandSolder
- R23: value 10k -> 1k; footprint Resistor_THT:R_Axial_DIN0207_L6.3mm_D2.5mm_P7.62mm_Horizontal -> Resistor_SMD:R_0805_2012Metric_Pad1.20x1.40mm_HandSolder
- R24: value 470R -> 330R; footprint Resistor_THT:R_Axial_DIN0207_L6.3mm_D2.5mm_P7.62mm_Horizontal -> Resistor_SMD:R_0805_2012Metric_Pad1.20x1.40mm_HandSolder
- R25: value 27k -> 20k; footprint Resistor_THT:R_Axial_DIN0207_L6.3mm_D2.5mm_P7.62mm_Horizontal -> Resistor_SMD:R_0805_2012Metric_Pad1.20x1.40mm_HandSolder
- R26: value 1k -> 10k; footprint Resistor_THT:R_Axial_DIN0207_L6.3mm_D2.5mm_P7.62mm_Horizontal -> Resistor_SMD:R_0805_2012Metric_Pad1.20x1.40mm_HandSolder
- R27: value 10k -> 5.6k; footprint Resistor_THT:R_Axial_DIN0207_L6.3mm_D2.5mm_P7.62mm_Horizontal -> Resistor_SMD:R_0805_2012Metric_Pad1.20x1.40mm_HandSolder
- R28: value 18k -> 1k; footprint Resistor_THT:R_Axial_DIN0207_L6.3mm_D2.5mm_P7.62mm_Horizontal -> Resistor_SMD:R_0805_2012Metric_Pad1.20x1.40mm_HandSolder
- R29: value 100k -> 25m (NOTA 1); footprint Resistor_THT:R_Axial_DIN0207_L6.3mm_D2.5mm_P7.62mm_Horizontal -> Resistor_SMD:R_2512_6332Metric
- R3: value 39K -> 180k; footprint Resistor_THT:R_Axial_DIN0207_L6.3mm_D2.5mm_P7.62mm_Horizontal -> Resistor_SMD:R_0805_2012Metric_Pad1.20x1.40mm_HandSolder
- R30: value 330k -> 4,7K; footprint Resistor_THT:R_Axial_DIN0207_L6.3mm_D2.5mm_P7.62mm_Horizontal -> Resistor_THT:R_Axial_DIN0922_L20.0mm_D9.0mm_P7.62mm_Vertical
- R31: value 4.7k -> 270k; footprint Resistor_THT:R_Axial_DIN0207_L6.3mm_D2.5mm_P7.62mm_Horizontal -> Resistor_SMD:R_0805_2012Metric_Pad1.20x1.40mm_HandSolder
- R32: value 4.7k -> 1k; footprint Resistor_THT:R_Axial_DIN0207_L6.3mm_D2.5mm_P7.62mm_Horizontal -> Resistor_SMD:R_0805_2012Metric_Pad1.20x1.40mm_HandSolder; moved to B.Cu
- R33: value 330k -> 220R; footprint Resistor_THT:R_Axial_DIN0207_L6.3mm_D2.5mm_P7.62mm_Horizontal -> Resistor_SMD:R_0805_2012Metric_Pad1.20x1.40mm_HandSolder; moved to B.Cu
- R34: value 330k -> 27k
- R35: value 27k -> 18k
- R36: value 47k -> 1k; footprint Resistor_THT:R_Axial_DIN0207_L6.3mm_D2.5mm_P7.62mm_Horizontal -> Resistor_SMD:R_0805_2012Metric_Pad1.20x1.40mm_HandSolder
- R37: value 470R -> 100k
- R38: value R -> 10R; footprint Resistor_THT:R_Axial_DIN0207_L6.3mm_D2.5mm_P7.62mm_Horizontal -> Resistor_SMD:R_0805_2012Metric_Pad1.20x1.40mm_HandSolder
- R39: value 100K -> 1k; footprint Resistor_THT:R_Axial_DIN0207_L6.3mm_D2.5mm_P7.62mm_Horizontal -> oxebots:Resistor_RX24_10W
- R4: value 39K -> 270k; footprint Resistor_THT:R_Axial_DIN0207_L6.3mm_D2.5mm_P7.62mm_Horizontal -> Resistor_SMD:R_0805_2012Metric_Pad1.20x1.40mm_HandSolder
- R40: value R -> 10k; footprint Resistor_THT:R_Axial_DIN0207_L6.3mm_D2.5mm_P7.62mm_Horizontal -> Resistor_SMD:R_0805_2012Metric_Pad1.20x1.40mm_HandSolder
- R41: value 4.7k -> 330k; footprint Resistor_THT:R_Axial_DIN0207_L6.3mm_D2.5mm_P7.62mm_Horizontal -> Resistor_SMD:R_0805_2012Metric_Pad1.20x1.40mm_HandSolder
- R42: value 4.7k -> 510k; footprint Resistor_THT:R_Axial_DIN0207_L6.3mm_D2.5mm_P7.62mm_Horizontal -> Resistor_THT:R_Axial_DIN0207_L6.3mm_D2.5mm_P15.24mm_Horizontal
- R5: value 10R -> 1k; footprint Resistor_THT:R_Axial_DIN0207_L6.3mm_D2.5mm_P7.62mm_Horizontal -> Resistor_SMD:R_0805_2012Metric_Pad1.20x1.40mm_HandSolder
- R6: value 25m (NOTA 1) -> 39K; footprint Resistor_SMD:R_2512_6332Metric -> Resistor_SMD:R_0805_2012Metric_Pad1.20x1.40mm_HandSolder
- R7: footprint Resistor_THT:R_Axial_DIN0207_L6.3mm_D2.5mm_P7.62mm_Horizontal -> Resistor_SMD:R_0805_2012Metric_Pad1.20x1.40mm_HandSolder
- R8: value 1,5K -> 10k; footprint Resistor_THT:R_Axial_DIN0207_L6.3mm_D2.5mm_P7.62mm_Horizontal -> Resistor_SMD:R_0805_2012Metric_Pad1.20x1.40mm_HandSolder
- R9: value 300k -> 10k; footprint Resistor_THT:R_Axial_DIN0207_L6.3mm_D2.5mm_P7.62mm_Horizontal -> Resistor_SMD:R_0805_2012Metric_Pad1.20x1.40mm_HandSolder
- U1: value LT3751 -> LM324; footprint Package_SO:TSSOP-20-1EP_4.4x6.5mm_P0.65mm_EP2.15x3.35mm -> Package_SO:SOIC-14_3.9x8.7mm_P1.27mm
- U2: value PC817 -> LMV358; footprint Package_DIP:DIP-4_W7.62mm -> Package_SO:SOIC-8_5.3x6.2mm_P1.27mm
- U3: value STM32F030F4Px -> TLV431DBZ; footprint Package_SO:TSSOP-20_4.4x6.5mm_P0.65mm -> Package_TO_SOT_SMD:SOT-23
- U4: value PC817 -> LT3751; footprint Package_DIP:DIP-4_W7.62mm -> Package_SO:TSSOP-20-1EP_4.4x6.5mm_P0.65mm_EP2.15x3.35mm
- U7: value LM358 -> HCPL-3120; footprint Package_DIP:DIP-8_W7.62mm -> Package_DIP:DIP-8_W7.62mm_LongPads
- U8: value HCNR201 -> LM358; footprint Package_DIP:DIP-8_W7.62mm_LongPads -> Package_SO:SOIC-8_5.3x6.2mm_P1.27mm
- moved RV1 226.4 mm to (58.4, 111.8), turned to 180 degrees
- moved C8 224.1 mm to (47.2, 129.1), turned to -90 degrees
- moved D4 208.1 mm to (69.5, 120.4), turned to 180 degrees
- moved R1 204.9 mm to (59.4, 121.4), turned to -90 degrees
- moved R14 195.8 mm to (43.9, 121.4), turned to 90 degrees
- moved C2 195.6 mm to (69.4, 90.2)
- moved R25 191.5 mm to (52.1, 100.1)
- moved C11 191.3 mm to (79.8, 132.9), turned to -90 degrees
- moved R26 190.1 mm to (52.1, 96.8), turned to 180 degrees
- moved R15 189.5 mm to (56.6, 140.0), turned to -90 degrees
- moved R23 188.3 mm to (58.9, 106.2), turned to 180 degrees
- moved J3 188.0 mm to (84.8, 88.2), turned to -90 degrees
- moved R29 185.6 mm to (62.2, 131.9), turned to 90 degrees
- moved R20 184.6 mm to (53.8, 140.0), turned to -90 degrees
- moved R11 184.3 mm to (39.7, 131.8), turned to -90 degrees
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Connections:
- C1 pad 1: +12V -> +24V
- C10 pad 1: LT3751_FB -> +12V
- C11 pad 1: +3.3V -> Net-(C11-Pad1)
- C11 pad 2: GND -> Net-(Q3-D)
- C12 pad 1: +3.3V -> VCAP
- C12 pad 2: GND -> GNDPWR
- C13 pad 1: +12V -> +15V_SEC
- C13 pad 2: GND -> GNDPWR
- C15 pad 1: +15V_SEC -> Net-(Q4-G)
- C16 pad 1: Net-(C16-Pad1) -> VCAP
- C16 pad 2: GND -> GNDPWR
- C17 pad 1: Net-(C17-Pad1) -> +15V_SEC
- C17 pad 2: GND -> GNDPWR
- C18 pad 1: +3.3V -> VCAP
- C18 pad 2: GND -> GNDPWR
- C19 pad 1: Net-(Q4-G) -> +15V_SEC
- C2 pad 1: +24V -> +3.3V
- C3 pad 1: +24V -> +12V
- C4 pad 1: VCAP -> +24V
- C4 pad 2: GNDPWR -> GND
- C5 pad 1: VCAP -> +12V
- C5 pad 2: GNDPWR -> GND
- C6 pad 1: VCAP -> +3.3V
- C6 pad 2: GNDPWR -> GND
- C7 pad 1: Net-(C7-Pad1) -> +12V
- C7 pad 2: Net-(Q1-D) -> GND
- C8 pad 1: +12V -> LT3751_FB
- C9 pad 1: +12V -> Net-(U1C--)
- C9 pad 2: GND -> Net-(U1B-+)
- D1 pad 1: GND -> VCAP
- D1 pad 2: +24V -> Net-(D1-A)
- D2 pad 1: VCAP -> Net-(D2-K)
- D2 pad 2: Net-(D2-A) -> GNDPWR
- D4 pad 1: VCAP -> +24V
- D4 pad 2: Net-(D4-A2) -> GND
- J2 pad 1: +24V -> +3.3V
- J2 pad 2: +24V -> GND
- J3 pad 1: +3.3V -> +12V
- Q1 pad 1: Net-(Q1-G) -> LT3751_DONE
- Q1 pad 2: Net-(Q1-D) -> GND
- Q1 pad 3: Net-(Q1-S) -> EXT_OUT_LT3751_DONE
- Q2 pad 1: Net-(Q2-G) -> LT3751_FAULT
- Q2 pad 2: Net-(D3-A2) -> GND
- Q2 pad 3: GNDPWR -> EXT_OUT_LT3751_FAULT
- Q3 pad 2: Net-(D4-A2) -> Net-(Q3-D)
- Q3 pad 3: GNDPWR -> Net-(Q3-S)
- Q5 pad 1: EXT_OUT_LT3751_DONE -> Net-(Q5-G)
- Q5 pad 2: LT3751_DONE -> Net-(D3-A2)
- Q5 pad 3: GND -> GNDPWR
- R1 pad 2: Net-(C7-Pad1) -> LT3751_UVLO_1
- R10 pad 1: +12V -> LT3751_FB
- R10 pad 2: UVLO_2 -> Net-(U3-REF)
- R11 pad 1: +24V -> Net-(U3-REF)
- R11 pad 2: OVLO_1 -> GND
- R12 pad 1: +12V -> Net-(U2A-+)
- R12 pad 2: OVLO_2 -> Net-(U1D--)
- R13 pad 1: +15V_SEC -> Net-(U2A-+)
- R13 pad 2: Net-(R13-Pad2) -> Net-(U2B--)
- R14 pad 1: EXT_IN_LT3751_KICK_1 -> LT3751_FB
- R14 pad 2: Net-(C16-Pad1) -> Net-(U1A--)
- R15 pad 1: MCU_OUT_KICK_1 -> Net-(U4-RBG)
- R15 pad 2: Net-(C16-Pad1) -> GND
- R16 pad 1: Net-(R13-Pad2) -> +3.3V
- R16 pad 2: Net-(Q2-G) -> LT3751_DONE
- R17 pad 1: Net-(Q2-G) -> +3.3V
- R17 pad 2: GNDPWR -> LT3751_FAULT
- R18 pad 1: +15V_SEC -> Net-(U4-RDCM)
- R18 pad 2: Net-(R18-Pad2) -> Net-(Q3-D)
- R19 pad 1: EXT_IN_LT3751_KICK_1 -> Net-(U4-RVOUT)
- R19 pad 2: Net-(C17-Pad1) -> Net-(Q3-D)
- R2 pad 1: Net-(U1-RDCM) -> +24V
- R2 pad 2: Net-(Q1-D) -> LT3751_OVLO_1
- R20 pad 1: MCU_OUT_KICK_2 -> Net-(U4-HVGATE)
- R20 pad 2: Net-(C17-Pad1) -> Net-(Q3-G)
- R21 pad 1: Net-(R18-Pad2) -> +3.3V
- R21 pad 2: Net-(Q3-G) -> EXT_OUT_LT3751_DONE
- R22 pad 1: Net-(Q3-G) -> +3.3V
- R22 pad 2: GNDPWR -> EXT_OUT_LT3751_FAULT
- R23 pad 1: +3.3V -> Net-(U1B--)
- R23 pad 2: MCU_RST -> Net-(U1A-+)
- R24 pad 1: MCU_OUT_BLEEDER -> Net-(R24-Pad1)
- R24 pad 2: Net-(R24-Pad2) -> GND
- R25 pad 1: Net-(R25-Pad1) -> Net-(U1B--)
- R25 pad 2: VCAP -> Net-(U1D-+)
- R26 pad 1: VCAP -> Net-(U1D-+)
- R26 pad 2: Net-(Q4-A) -> GND
- R27 pad 1: MCU_OUT_BLEEDER -> +3.3V
- R27 pad 2: GND -> Net-(U2B-+)
- R28 pad 1: Net-(D5-K) -> Net-(U2B-+)
- R28 pad 2: Net-(Q4-G) -> GND
- R29 pad 1: Net-(Q4-G) -> Net-(Q3-S)
- R29 pad 2: GNDPWR -> GND
- R3 pad 1: Net-(U1-RVOUT) -> +12V
- R3 pad 2: Net-(Q1-D) -> LT3751_UVLO_2
- R30 pad 1: VCAP -> +24V
- R30 pad 2: Net-(R30-Pad2) -> Net-(C11-Pad1)
- R31 pad 1: +3.3V -> Net-(R31-Pad1)
- R31 pad 2: LT3751_DONE -> Net-(U1C--)
- R32 pad 1: +3.3V -> +12V
- R32 pad 2: EXT_OUT_LT3751_DONE -> Net-(R32-Pad2)
- R33 pad 1: Net-(R30-Pad2) -> EXT_IN_LT3751_KICK_1
- R33 pad 2: Net-(R33-Pad2) -> Net-(U7-A)
- R34 pad 1: Net-(R33-Pad2) -> Net-(R34-Pad1)
- R34 pad 2: Net-(D6-K) -> VCAP
- R35 pad 1: Net-(R35-Pad1) -> Net-(D2-K)
- R35 pad 2: Net-(U6A--) -> Net-(Q4-G)
- R36 pad 1: Net-(U7B--) -> Net-(R36-Pad1)
- R36 pad 2: Net-(U7A--) -> Net-(R36-Pad2)
- R37 pad 1: Net-(R37-Pad1) -> Net-(Q4-G)
- R37 pad 2: Net-(R37-Pad2) -> GNDPWR
- R38 pad 1: Net-(U6C-+) -> Net-(R38-Pad1)
- R38 pad 2: Net-(U6B-+) -> Net-(Q5-G)
- R39 pad 1: Net-(D6-K) -> VCAP
- R39 pad 2: GNDPWR -> Net-(Q4-A)
- R4 pad 1: +24V -> +12V
- R4 pad 2: Net-(U1-RVTRANS) -> LT3751_OVLO_2
- R40 pad 1: Net-(U6B-+) -> Net-(Q5-G)
- R40 pad 2: Net-(R40-Pad2) -> GNDPWR
- R41 pad 1: +3.3V -> Net-(U8A--)
- R41 pad 2: LT3751_FAULT -> Net-(U8B--)
- R42 pad 1: +3.3V -> VCAP
- R42 pad 2: EXT_OUT_LT3751_FAULT -> Net-(R42-Pad2)
- R5 pad 1: Net-(U1-HVGATE) -> EXT_OUT_FB
- R5 pad 2: Net-(Q1-G) -> Net-(R5-Pad2)
- R6 pad 1: Net-(Q1-S) -> +24V
- R6 pad 2: GND -> Net-(U4-RVTRANS)
- R7 pad 1: MCU_OUT_ENABLE -> EXT_IN_LT3751_ENABLE
- R7 pad 2: Net-(U1-CHARGE) -> Net-(U4-CHARGE)
- R8 pad 1: Net-(U1-RBG) -> Net-(R5-Pad2)
- R8 pad 2: GND -> Net-(U2A--)
- R9 pad 1: +24V -> Net-(U2A--)
- R9 pad 2: UVLO_1 -> GND
- RV1 pad 1: Net-(R35-Pad1) -> Net-(U1A-+)
- RV1 pad 2: Net-(R40-Pad2) -> Net-(R24-Pad1)
- RV1 pad 3: Net-(R40-Pad2) -> Net-(R24-Pad1)
- T1 pad 1: Net-(D2-A) -> Net-(D1-A)
- T1 pad 6: Net-(Q1-D) -> Net-(Q3-D)
- T1 pad 7: Net-(Q1-D) -> Net-(Q3-D)
- U1 pad 1: Net-(U1-RVTRANS) -> Net-(U1A--)
- U1 pad 10: LT3751_FB -> GND
- U1 pad 12: Net-(Q1-S) -> Net-(U1D-+)
- U1 pad 13: +12V -> Net-(U1D--)
- U1 pad 14: +12V -> Net-(U1D--)
- U1 pad 2: LT3751_UVLO_1 -> Net-(U1A--)
- U1 pad 3: LT3751_OVLO_1 -> Net-(U1A-+)
- U1 pad 4: LT3751_UVLO_2 -> +12V
- U1 pad 5: LT3751_OVLO_2 -> Net-(U1B-+)
- U1 pad 6: LT3751_FAULT -> Net-(U1B--)
- U1 pad 7: LT3751_DONE -> Net-(U1B--)
- U1 pad 8: Net-(U1-CHARGE) -> Net-(U1B-+)
- U1 pad 9: GND -> Net-(U1C--)
- U2 pad 1: Net-(C16-Pad1) -> Net-(R5-Pad2)
- U2 pad 2: GND -> Net-(U2A--)
- U2 pad 3: GNDPWR -> Net-(U2A-+)
- U2 pad 4: Net-(R13-Pad2) -> GND
- U3 pad 1: unconnected-(U3-BOOT0-Pad1) -> LT3751_FB
- U3 pad 2: unconnected-(U3-PF0-Pad2) -> Net-(U3-REF)
- U3 pad 3: unconnected-(U3-PF1-Pad3) -> GND
- U4 pad 1: Net-(C17-Pad1) -> Net-(U4-RVTRANS)
- U4 pad 2: GND -> LT3751_UVLO_1
- U4 pad 3: GNDPWR -> LT3751_OVLO_1
- U4 pad 4: Net-(R18-Pad2) -> LT3751_UVLO_2
- U7 pad 1: Net-(U7A--) -> unconnected-(U7-NC-Pad1)
- U7 pad 2: Net-(U7A--) -> Net-(U7-A)
- U7 pad 3: Net-(D6-K) -> GND
- U7 pad 4: GNDPWR -> unconnected-(U7-NC-Pad4)
- U7 pad 6: Net-(U7B--) -> Net-(R38-Pad1)
- U7 pad 7: Net-(R37-Pad2) -> Net-(R38-Pad1)
- U8 pad 1: Net-(R37-Pad1) -> Net-(R36-Pad2)
- U8 pad 2: +15V_SEC -> Net-(U8A--)
- U8 pad 3: Net-(U7B--) -> GNDPWR
- U8 pad 5: GND -> Net-(U8B-+)
- U8 pad 6: Net-(U6A--) -> Net-(U8B--)
- U8 pad 7: unconnected-(U8-Pad7) -> Net-(U8B--)
- U8 pad 8: unconnected-(U8-Pad8) -> +15V_SEC
Routing:
- net LT3751_DONE: track 0.00 -> 49.3 mm
- net LT3751_FAULT: track 0.00 -> 48.2 mm
- net +15V_SEC: track 0.00 -> 46.3 mm
- net Net-(U1C--): track 0.00 -> 37.9 mm
- net +3.3V: track 0.00 -> 34.6 mm
- net +12V: track 0.00 -> 33.7 mm
- net Net-(U1B--): track 0.00 -> 26.9 mm
- net Net-(U1B-+): track 0.00 -> 21.3 mm, vias 0 -> 1
- net GNDPWR: track 0.00 -> 20.7 mm
- net Net-(R5-Pad2): track 0.00 -> 19.9 mm
- net Net-(Q4-G): track 0.00 -> 19.1 mm
- net Net-(U2A-+): track 0.00 -> 18.1 mm, vias 0 -> 2
- net Net-(U8B--): track 0.00 -> 16.9 mm
- net EXT_OUT_LT3751_FAULT: track 0.00 -> 15.4 mm
- net Net-(U1D--): track 0.00 -> 15.0 mm
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- added copper zone on B.Cu, net GNDPWR
- added copper zone on F.Cu, net GNDPWR
- added copper zone on F.Cu, net Net-(C11-Pad1)
- added copper zone on F.Cu, net Net-(D1-A)
- added copper zone on F.Cu, net Net-(D3-A2)
- added copper zone on F.Cu, net Net-(Q3-D)
- added copper zone on F.Cu, net Net-(Q3-S)
- added copper zone on F.Cu, net Net-(Q4-A)
- added copper zone on F.Cu, net VCAP
Other:
- outline, holes or cut-outs redrawn
