File: pcbs/kicker/Kicker_LT3751_OxeBots.kicad_sch (KiCad schematic)
At the start: 75 parts, among them J1 POWER, J2 POWER, J3 REG_12V, J5 SOL, Q1 IRFB4227, Q2 FGH60N60SMD, SW1 SW_Push, T1 DCT15EFD-U44S003, U2 LM7805_TO220, U3 HCPL-3120, U4 LM324

Commit message: First commit of Kicker Board
Parts:
- removed C11, C8: 100nF, Capacitor_THT:C_Disc_D5.0mm_W2.5mm_P2.50mm, symbol Device:C
- removed C3: 10nF, Capacitor_THT:C_Disc_D5.0mm_W2.5mm_P2.50mm, symbol Device:C
- removed C7: 1000uF, Capacitor_THT:CP_Radial_D8.0mm_P5.00mm, symbol Device:C_US
- removed D2: MUR460, Diode_THT:D_DO-201AD_P12.70mm_Horizontal, symbol Device:D
- removed D3, D4, D5: LED, LED_THT:LED_D3.0mm_Clear, symbol Device:LED
- removed IC?: LT3751, cusf:TSSOP-20-EP, symbol LT3751:LT3751
- removed J1, J2: POWER, TerminalBlock_Phoenix:TerminalBlock_Phoenix_MKDS-1,5-2_1x02_P5.00mm_Horizontal, symbol Connector:Screw_Terminal_01x02
- removed J3: REG_12V, Connector_PinSocket_2.54mm:PinSocket_1x04_P2.54mm_Vertical, symbol Connector:Conn_01x04_Socket
- removed J4: ~, Connector_PinHeader_2.54mm:PinHeader_1x06_P2.54mm_Vertical, symbol Connector:Conn_01x06_Pin
- removed J5: SOL, TerminalBlock_Phoenix:TerminalBlock_Phoenix_MKDS-1,5-2_1x02_P5.00mm_Horizontal, symbol Connector:Screw_Terminal_01x02
- removed JP1, JP2, JP3, JP4: ~, Jumper:SolderJumper-2_P1.3mm_Open_Pad1.0x1.5mm, symbol Jumper:Jumper_2_Open
- removed Q2: FGH60N60SMD, Package_TO_SOT_THT:TO-247-3_Vertical, symbol Device:Q_NIGBT_GCE
- removed R13: 510K, Resistor_THT:R_Axial_DIN0207_L6.3mm_D2.5mm_P7.62mm_Horizontal, symbol Device:R
- removed R16: 220K, Resistor_THT:R_Axial_DIN0207_L6.3mm_D2.5mm_P7.62mm_Horizontal, symbol Device:R
- removed R17: 220R, Resistor_THT:R_Axial_DIN0207_L6.3mm_D2.5mm_P7.62mm_Horizontal, symbol Device:R
- removed R18: R, Resistor_THT:R_Axial_DIN0207_L6.3mm_D2.5mm_P7.62mm_Horizontal, symbol Device:R
- removed T1: DCT15EFD-U44S003, oxebots_transformer:TRANS_U44S003_TDK, symbol DCT15EFD_U44S003:DCT15EFD-U44S003
- removed U2: LM7805_TO220, Package_TO_SOT_THT:TO-220-3_Vertical, symbol Regulator_Linear:LM7805_TO220
- removed U3: HCPL-3120, Package_DIP:DIP-8_W7.62mm, symbol Driver_FET:HCPL-3120
- removed U4: LM324, Package_DIP:DIP-14_W7.62mm, symbol Amplifier_Operational:LM324
- added C11, C15, C8: 220uF, Capacitor_THT:CP_Radial_D8.0mm_P5.00mm, symbol Device:C_US
- added C19, C20, C21, C23, C24, C25, C9: 100nF, Capacitor_THT:C_Disc_D5.0mm_W2.5mm_P2.50mm, symbol Device:C
- added C22: C, symbol Device:C
- added C6: 820uF, Capacitor_THT:CP_Radial_D30.0mm_P10.00mm_SnapIn, symbol Device:C_US
- added D1: SMBJ26A, symbol Device:D_TVS
- added D3, D4: MUR460, Diode_THT:D_DO-201AD_P12.70mm_Horizontal, symbol Device:D
- added D5: D_Zener, symbol Device:D_Zener
- added F1: 10A, symbol Device:Fuse
- added J1, J6, J7: XT30PW-F, XT30PW-F:AMASS_XT30PW-F, symbol oxebots:XT30PW-F
- added J2, J3: CONN_BUCK, symbol Connector:Conn_01x04_Pin
- added J4: EXT UART, symbol Connector:Conn_01x04_Pin
- added J5: Programmer, symbol Connector:Conn_01x05_Pin
- added JP1: ~, symbol Jumper:SolderJumper_3_Open
- added PS1: B1205S, Converter_DCDC:Converter_DCDC_Murata_MEE1SxxxxSC_THT, symbol Converter_DCDC:MEE1S1515SC
- added Q2, Q4: BC547, Package_TO_SOT_THT:TO-92_Inline, symbol Transistor_BJT:BC547
- added Q3, Q5: FGH60N60SMD, Package_TO_SOT_THT:TO-247-3_Vertical, symbol Device:Q_NIGBT_GCE
- added Q6: TIC106, Package_TO_SOT_THT:TO-220-3_Vertical, symbol Triac_Thyristor:TIC106
- added R26: R, Resistor_THT:R_Axial_DIN0207_L6.3mm_D2.5mm_P7.62mm_Horizontal, symbol Device:R
- added R28: 10k, symbol Device:R
- added R30: 27k, symbol Device:R
- added R34: 18k, symbol Device:R
- added T1: DCT15EFD-U44S003, TDK DCT15EFD-U44S003:TRANS_U44S003_TDK, symbol oxebots:DCT15EFD-U44S003
- added U1: LT3751, cusf:TSSOP-20-EP, symbol oxebots:LT3751
- added U2: ISO1540, Package_SO:SOIC-8_3.9x4.9mm_P1.27mm, symbol Isolator:ISO1540
- added U3: ADS1115IDGS, Package_SO:TSSOP-10_3x3mm_P0.5mm, symbol Analog_ADC:ADS1115IDGS
- added U4: STM32F070F6P6, Package_SO:TSSOP-20_4.4x6.5mm_P0.65mm, symbol MCU_ST_STM32F0:STM32F070F6Px
- added U5, U7: HCPL-3120, Package_DIP:DIP-8_W7.62mm, symbol Driver_FET:HCPL-3120
- added U6: STM32F103C8Tx, Package_QFP:LQFP-48_7x7mm_P0.5mm, symbol MCU_ST_STM32F1:STM32F103C8Tx
- added U8: AQV453, RELAY_AQV_DIP6_25X_PAN, symbol oxebots:AQV453
- added U9: TLV9001IDCK, Package_TO_SOT_SMD:SOT-353_SC-70-5, symbol Amplifier_Operational:TLV9001IDCK
- C14: value C -> 100nF
- C4: value 10nF -> 100nF
- C5: value 100uF -> 820uF
- R10: value ? -> 180k; footprint Resistor_THT:R_Axial_DIN0207_L6.3mm_D2.5mm_P7.62mm_Horizontal -> (none)
- R11: value ? -> 510k; footprint Resistor_THT:R_Axial_DIN0207_L6.3mm_D2.5mm_P7.62mm_Horizontal -> (none)
- R12: value 1M -> 270k; footprint Resistor_THT:R_Axial_DIN0207_L6.3mm_D2.5mm_P7.62mm_Horizontal -> (none)
- R13: renamed from R26; value R -> 330k
- R14: value 360K -> 330k
- R15: value 300K -> 330k
- R16: renamed from R28; value R -> 100K
- R17: renamed from R30; value 10K -> 4.7k
- R18: renamed from R34; value 1K -> 4.7k
- R19: value R -> 220R
- R21: value 47K -> R
- R22: value R -> 4.7k
- R23: value 10K -> 4.7k
- R24: value 1K -> 220R
- R25: value 15K -> R
- R27, R33: value 10K -> R; footprint Resistor_THT:R_Axial_DIN0207_L6.3mm_D2.5mm_P7.62mm_Horizontal -> (none)
- R29: value 10K -> 470R; footprint Resistor_THT:R_Axial_DIN0207_L6.3mm_D2.5mm_P7.62mm_Horizontal -> (none)
- R31: value 10K -> 1k; footprint Resistor_THT:R_Axial_DIN0207_L6.3mm_D2.5mm_P7.62mm_Horizontal -> (none)
- R32: value 10K -> 10k; footprint Resistor_THT:R_Axial_DIN0207_L6.3mm_D2.5mm_P7.62mm_Horizontal -> (none)
- R35: value 1K -> 100k; footprint Resistor_THT:R_Axial_DIN0207_L6.3mm_D2.5mm_P7.62mm_Horizontal -> (none)
- R8: value 1,5K (NOTA 2) -> 1,5K
- R9: value ? -> 300k; footprint Resistor_THT:R_Axial_DIN0207_L6.3mm_D2.5mm_P7.62mm_Horizontal -> (none)
- SW1: footprint Button_Switch_THT:SW_PUSH_6mm_H7.3mm -> (none)
- renumbered C9 to C1, C15 to C16, C16 to C17, C17 to C18, C1 to C2, C2 to C3, C6 to C7, D1 to D2, PS1 to PS2, R3 to R2, R4 to R3, R2 to R4
Connections:
- net MCU_OUT_DONE is gone; now on net GND: R32.2
- net +12V: now also C13.1, R10.1, R12.1, C8.1, C9.1, J2.3 (Pin_3), PS1.2 (+Vin), U1.13 (VCC), U1.14 (LVGATE); no longer R14.1
- net +15V_SEC: now also U5.8 (VCC), U7.8 (VCC)
- net +24V: now also R11.1, R9.1, D1.2 (A2), F1.2, J2.1 (Pin_1), J2.2 (Pin_2), J3.1 (Pin_1), J3.2 (Pin_2), T1.4, T1.5; no longer R15.1
- net GND: now also C11.2, C19.2, C20.2, C21.2, C23.2, C24.2, C8.2, C9.2, D1.1 (A1), J1.N, J2.4 (Pin_4), J3.4 (Pin_4), J4.4 (Pin_4), J5.5 (Pin_5), JP1.3 (B), PS1.1 (-Vin), Q2.3 (E), Q4.3 (E), U1.11 (CSN), U1.21 (GND), U1.9 (CLAMP), U2.4 (GND1), U4.15 (VSS), U5.3 (C), U7.3 (C), U8.2, U9.1 (+), U9.2 (V-); no longer C14.2, C17.2, C18.2, C4.2, C5.2, PS2.3 (-Vout), R12.2, R16.2, R19.2, R25.2, R29.2
- net OVLO_1: now also R11.2
- net OVLO_2: now also R12.2; no longer R14.2
- net UVLO_1: now also R9.2; no longer R15.2
- net UVLO_2: now also R10.2
- net VCAP: now also R31.1, C6.1, D3.1 (K), D4.1 (K), J6.P, J7.P, R30.2; no longer R10.1, R11.1, R12.1, R9.1
- net at R8.1: now also U1.16 (RBG)
- net MCU_OUT_KICK_1: now reaches R19.1
- net MCU_OUT_KICK_1: now also U4.6 (PA0)
- net at R3.1: now also U1.18 (RVOUT)
- net at C7.2, Q1.2 (D), R2.2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: now also T1.6, T1.7
- net +3.3V: now reaches R18.1
- net +3.3V: now also C12.1, R17.1, R22.1, R23.1, C11.1, C19.1, C23.1, C24.1, J3.3 (Pin_3), J4.1 (Pin_1), J5.1 (Pin_1), JP1.1 (A), R28.1, U2.1 (VCC1), U4.16 (VDD), U4.5 (VDDA), U9.5 (V+); no longer R32.1
- net MCU_IN_DONE: now reaches R18.2
- net MCU_IN_DONE: now also Q2.1 (C), U4.11 (PA5)
- net at R20.1: now also U5.6 (VO), U5.7 (VO); no longer R22.2
- net at R25.1: now also U7.6 (VO), U7.7 (VO); no longer R21.2
- net at R24.2: now also C21.1, U7.2 (A)
- net at R5.1: now also U1.15 (HVGATE)
- net at R7.2: now also U1.8 (CHARGE)
- net at Q1.3 (S), R6.1: now also U1.12 (CSP)
- net at R4.2: now also U1.1 (RVTRANS)
- net at R35.1: now also C25.1, Q6.3 (G), R34.2; no longer R33.1
- net at D2.2 (A): now also T1.1
- net GNDPWR: now reaches R35.2
- net GNDPWR: now also C14.2, C17.2, C18.2, C4.2, C5.2, PS2.3 (-Vout), R16.2, R21.2, C15.2, C25.2, C6.2, D5.2 (A), PS1.3 (-Vout), Q3.3 (E), Q5.3 (E), Q6.1 (K), R26.2, T1.10, U2.5 (GND2), U3.3 (GND), U5.5 (VEE), U7.5 (VEE)
- net at R2.1: now also U1.20 (RDCM)
- removed net +5V: C12.1, C14.1, R17.1, R21.1, R27.1, R31.1
- net DONE renamed LT3751_DONE
- net LT3751_DONE: now also Q2.2 (B), U1.7 (~{DONE})
- net FAULT: no longer names the net of R31.2
- net FAULT: now also Q6.2 (A)
- removed net FB: C10.1, R13.2, R16.1
- net MCU_IN_ENABLE renamed MCU_OUT_ENABLE
- net MCU_OUT_ENABLE: now also U4.13 (PA7)
- net MCU_OUT_CAP renamed MCU_IN_FAULT
- net MCU_IN_FAULT: now also Q4.1 (C), U4.10 (PA4)
- net MCU_OUT_FAULT: no longer names the net of R33.2
- net MCU_OUT_FAULT: now also R27.1, C22.1, U9.3 (-)
- net VREF renamed LT3751_FB
- net LT3751_FB: now also C10.1, C22.2, U1.10 (FB), U9.4; no longer R29.1
- new net: R14.2, R15.1
- new net: R15.2, R16.1, U3.4 (AIN0)
- new net: R29.2, U8.1
- new net: F1.1, J1.P
- new net: C20.1, R19.2, U5.2 (A)
- new net: Q5.1 (G), R25.2, R26.1
- new net: D5.1 (K), R34.1, U8.4
- new net: R13.2, R14.1
- new net: R30.1, U8.6
- new net: U2.6 (SCL2), U3.10 (SCL)
- new net: U2.7 (SDA2), U3.9 (SDA)
- new net: D4.2 (A), J7.N, Q5.2 (C)
- new net: Q3.1 (G), R20.2, R21.1
- new net: D3.2 (A), J6.N, Q3.2 (C)
- new net: U6.23 (VSS), U6.35 (VSS), U6.47 (VSS)
- new net +5V_SEC: C14.1, C15.1, PS1.4 (+Vout), U2.8 (VCC2), U3.8 (VDD)
- new net EXT_MCU_RX: J4.3 (Pin_3), U4.9 (PA3)
- new net EXT_MCU_TX: J4.2 (Pin_2), U4.8 (PA2)
- new net LT3751_FAULT: Q4.2 (B), R22.2, U1.6 (~{FAULT})
- new net LT3751_OVLO_1: U1.3 (OVLO1)
- new net LT3751_OVLO_2: U1.5 (OVLO2)
- new net LT3751_UVLO_1: U1.2 (UVLO1)
- new net LT3751_UVLO_2: U1.4 (UVLO2)
- new net MCU_BOOT0: JP1.2 (C), U4.1 (BOOT0)
- new net MCU_I2C_SCL: U2.3 (SCL1), U4.17 (PA9/PA11)
- new net MCU_I2C_SDA: U2.2 (SDA1), U4.18 (PA10/PA12)
- new net MCU_OUT_BLEEDER: R29.1, R32.1, U4.14 (PB1)
- new net MCU_OUT_FB: R33.1, U4.12 (PA6)
- new net MCU_OUT_KICK_2: R24.1, U4.7 (PA1)
- new net MCU_RST: J5.2 (Pin_2), R28.2, SW1.2, U4.4 (NRST)
- new net MCU_SWCLK: J5.4 (Pin_4), U4.20 (PA14)
- new net MCU_SWDIO: J5.3 (Pin_3), U4.19 (PA13)
- no-connect marks 1 -> 7
Other:
- note added: "+12V Power"
- note added: "+24V Power"
- note added: "+3.3V Power"
- note added: "1. +24V é fornecido por um pack Li-Ion 6S. A alimentação pode variar entre 16.8 e 25.2V. 2. R18 deve ter encapsulamento 1205. A resistência deve ser escolhida de acordo com a corrente máxima no primário do transformador, conforme relação a seguir. A potência do resistor deve ser acima da potência máxima dissipada, descrita abaixo: * 50 mOhms (R025): 2,1 A 0,2 W * 25 mOhms (R025): 4,2 A 0,4 W * 20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"
- note added: "50W Com dissipador"
- note added: "5W"
- note added: "Automatic Bleeder"
- note added: "DONE and FAULT Signal Conditioning"
- note added: "Digital Feedback Circuit"
- note added: "External Interfaces"
- note added: "External Programmer (ST Link)"
- note added: "External UART"
- note added: "High Voltage"
- note added: "Isolated Power +5V e +15V"
- note added: "Low-Pass Active Feedback Filter"
- note added: "Main Circuit"
- note added: "Microcontroller STM32"
- note added: "Power Circuits"
- note added: "Solenoid Circuit"
- note added: "Undervoltage and Overvoltage LT3751 Detection"
- note removed: "1. RX deve ter encapsulamento 1205. A resistência deve ser escolhida de acordo com a corrente máxima no primário do transformador, conforme relação a seguir. A potência do resistor deve ser acima da potência máxima dissipada, descrita abaixo: * 50 mOhms (R025): 2,1 A 0,2 W * 25 mOhms (R025): 4,2 A 0,4 W * 20 mOhms (R020): 5,3 A 0,6 W * 15 mOhms (R015): 7,1 A 0,7 W * 12 mOhms (R012): 8,8 A 0,9 W *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"
- note removed: "Acionamento do Solenoide"
- note removed: "Alta Tensão"
- note removed: "Baixa Tensão"
- note removed: "Bleeder de emergência"
- note removed: "Circuito de Bleeder"
- note removed: "Comparadores de sinal"
- note removed: "Feedback Isolado do Secundário"
- note removed: "Fonte Isolada +15V para o secundário"
- note removed: "Proteções contra sobretensão e subtensão"
- moved on the sheet: C1, C10, C16, C17, C18, C2, C3, C4, C5, C7, D2, PS2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

Commit message: Updated Solenoid Circuit
Parts:
- removed D3, D4: MUR460, Diode_THT:D_DO-201AD_P12.70mm_Horizontal, symbol Device:D
- removed Q3, Q5: FGH60N60SMD, Package_TO_SOT_THT:TO-247-3_Vertical, symbol Device:Q_NIGBT_GCE
- removed R24: 220R, Resistor_THT:R_Axial_DIN0207_L6.3mm_D2.5mm_P7.62mm_Horizontal, symbol Device:R
- removed U5, U7: HCPL-3120, Package_DIP:DIP-8_W7.62mm, symbol Driver_FET:HCPL-3120
- added D3, D4: 1.5KE300A, Diode_THT:D_DO-201AE_P15.24mm_Horizontal, symbol Diode:1.5KExxA
- added Q3, Q5: CS20N60, symbol Transistor_FET:Q_NMOS_GDS
- added R19, R25: 3.3k, Resistor_THT:R_Axial_DIN0207_L6.3mm_D2.5mm_P7.62mm_Horizontal, symbol Device:R
- added R26: 220R, Resistor_THT:R_Axial_DIN0207_L6.3mm_D2.5mm_P7.62mm_Horizontal, symbol Device:R
- added U6, U7: PC817, Package_DIP:DIP-4_W7.62mm, symbol Isolator:PC817
- R21: renamed from R20; value R -> 220R
- R22: renamed from R21; value R -> 3.3k
- R27: renamed from R25; value R -> 220R
- R28: renamed from R26; value R -> 3.3k
- renumbered R19 to R20, R22 to R23, R23 to R24, R27 to R29, R28 to R30, R29 to R31, R30 to R32, R31 to R33, R32 to R34, R33 to R35, R34 to R36, R35 to R37, U6 to U5
Connections:
- net +15V_SEC: now also R19.1, R25.1
- net GND: now also U6.2, U7.2
- net GNDPWR: now also Q3.3 (S), Q5.3 (S), U6.3, U7.3
- net MCU_OUT_KICK_2: now also R26.1
- net VCAP: now also D3.1 (A1), D4.1 (A1)
- net at C20.1, R20.2: now also U6.1
- net at R27.1: now also R25.2, U7.4
- net at R27.2, R28.1: now also Q5.1 (G)
- net at R21.1: now also R19.2, U6.4
- net at J7.N: now also D4.2 (A2), Q5.2 (D)
- net at C21.1: now also R26.2, U7.1
- net at R21.2, R22.1: now also Q3.1 (G)
- net at J6.N: now also D3.2 (A2), Q3.2 (D)
Other:
- moved on the sheet: C20, R20

Commit message: Updated feedback circuit
Parts:
- removed C13, C14, C19: 100nF, Capacitor_THT:C_Disc_D5.0mm_W2.5mm_P2.50mm, symbol Device:C
- removed C15: 220uF, Capacitor_THT:CP_Radial_D8.0mm_P5.00mm, symbol Device:C_US
- removed D5: D_Zener, symbol Device:D_Zener
- removed J3: CONN_BUCK, symbol Connector:Conn_01x04_Pin
- removed J4: EXT UART, symbol Connector:Conn_01x04_Pin
- removed J5: Programmer, symbol Connector:Conn_01x05_Pin
- removed PS1: B1205S, Converter_DCDC:Converter_DCDC_Murata_MEE1SxxxxSC_THT, symbol Converter_DCDC:MEE1S1515SC
- removed R29, R35: R, symbol Device:R
- removed U2: ISO1540, Package_SO:SOIC-8_3.9x4.9mm_P1.27mm, symbol Isolator:ISO1540
- removed U3: ADS1115IDGS, Package_SO:TSSOP-10_3x3mm_P0.5mm, symbol Analog_ADC:ADS1115IDGS
- removed U4: STM32F070F6P6, Package_SO:TSSOP-20_4.4x6.5mm_P0.65mm, symbol MCU_ST_STM32F0:STM32F070F6Px
- removed U5: STM32F103C8Tx, Package_QFP:LQFP-48_7x7mm_P0.5mm, symbol MCU_ST_STM32F1:STM32F103C8Tx
- removed U9: TLV9001IDCK, Package_TO_SOT_SMD:SOT-353_SC-70-5, symbol Amplifier_Operational:TLV9001IDCK
- added C16, C17: 100nF, Capacitor_THT:C_Disc_D5.0mm_W2.5mm_P2.50mm, symbol Device:C
- added C24: 100nF, Capacitor_THT:C_Rect_L19.0mm_W6.0mm_P15.00mm_MKS4, symbol Device:C
- added D4: 1.5KE300A, Diode_THT:D_DO-201AE_P15.24mm_Horizontal, symbol Diode:1.5KExxA
- added D6: 1N4712A, Diode_THT:D_DO-41_SOD81_P10.16mm_Horizontal, symbol Diode:1N47xxA
- added D7: SMBJ5.0A, Diode_SMD:D_SMB, symbol Diode:SMAJ5.0A
- added J3: Conn_01x02, Connector_JST:JST_XH_B2B-XH-A_1x02_P2.50mm_Vertical, symbol Connector_Generic:Conn_01x02
- added J5: XT30PW-F, oxebots_connectors:AMASS_XT30PW-M, symbol oxebots:XT30PW-F
- added J6: Conn_01x04, Connector_PinHeader_2.54mm:PinHeader_1x04_P2.54mm_Vertical, symbol Connector_Generic:Conn_01x04
- added J8: Conn_01x05, Connector_PinHeader_2.54mm:PinHeader_1x05_P2.54mm_Vertical, symbol Connector_Generic:Conn_01x05
- added J9: Conn_01x08, Connector_PinHeader_2.54mm:PinHeader_1x08_P2.54mm_Vertical, symbol Connector_Generic:Conn_01x08
- added Q3: FQD20N60, Package_TO_SOT_SMD:TO-263-2, symbol Transistor_FET:Q_NMOS_GDS
- added R14, R15, R22: 220R, Resistor_THT:R_Axial_DIN0207_L6.3mm_D2.5mm_P7.62mm_Horizontal, symbol Device:R
- added R18: 10R, Resistor_THT:R_Axial_DIN0207_L6.3mm_D2.5mm_P7.62mm_Horizontal, symbol Device:R
- added R20: 10k, Resistor_THT:R_Axial_DIN0207_L6.3mm_D2.5mm_P7.62mm_Horizontal, symbol Device:R
- added R38: 27k, Resistor_THT:R_Axial_DIN0207_L6.3mm_D2.5mm_P7.62mm_Horizontal, symbol Device:R
- added R39: 47k, Resistor_THT:R_Axial_DIN0207_L6.3mm_D2.5mm_P7.62mm_Horizontal, symbol Device:R
- added R40: 470R, Resistor_THT:R_Axial_DIN0207_L6.3mm_D2.5mm_P7.62mm_Horizontal, symbol Device:R
- added R41, R43: R, Resistor_THT:R_Axial_DIN0207_L6.3mm_D2.5mm_P7.62mm_Horizontal, symbol Device:R
- added RV1: 100k, Potentiometer_THT:Potentiometer_Bourns_3296W_Vertical, symbol Device:R_Potentiometer_Trim
- added U2: HCPL-3120, Package_DIP:DIP-8_W7.62mm, symbol Driver_FET:HCPL-3120
- added U4: STM32F030F4Px, Package_SO:TSSOP-20_4.4x6.5mm_P0.65mm, symbol MCU_ST_STM32F0:STM32F030F4Px
- added U7: LMF324, symbol Amplifier_Operational:LM324
- added U8: LM358, Package_DIP:DIP-8_W7.62mm, symbol Amplifier_Operational:LM358
- added U9: HCNR201, Package_DIP:DIP-8_W7.62mm_LongPads, symbol oxebots:HCNR201
- C22: footprint (none) -> Capacitor_THT:C_Disc_D5.0mm_W2.5mm_P2.50mm
- C23: footprint Capacitor_THT:C_Disc_D5.0mm_W2.5mm_P2.50mm -> Capacitor_THT:C_Rect_L19.0mm_W6.0mm_P15.00mm_MKS4
- D1: footprint (none) -> Diode_SMD:D_SMB_Handsoldering
- F1: footprint (none) -> Fuse:Fuse_Blade_ATO_directSolder
- J1, J7: footprint XT30PW-F:AMASS_XT30PW-F -> oxebots_connectors:AMASS_XT30PW-M
- J2: footprint (none) -> Connector_PinSocket_2.54mm:PinSocket_1x04_P2.54mm_Vertical
- J4: renamed from J6; footprint XT30PW-F:AMASS_XT30PW-F -> oxebots_connectors:AMASS_XT30PW-M
- JP1: footprint (none) -> Jumper:SolderJumper-3_P1.3mm_Open_Pad1.0x1.5mm
- Q2: renamed from Q3; footprint (none) -> Package_TO_SOT_SMD:TO-263-2
- Q4: renamed from Q5; footprint (none) -> Package_TO_SOT_SMD:TO-263-2
- R10, R11, R12, R9: footprint (none) -> Resistor_THT:R_Axial_DIN0207_L6.3mm_D2.5mm_P7.62mm_Horizontal
- R26: renamed from R30; footprint (none) -> Resistor_THT:R_Axial_DIN0207_L6.3mm_D2.5mm_P7.62mm_Horizontal
- R27: renamed from R31; footprint (none) -> Resistor_THT:R_Axial_DIN0207_L6.3mm_D2.5mm_P7.62mm_Horizontal
- R28: renamed from R32; footprint (none) -> Resistor_THT:R_Axial_DIN0207_L6.3mm_D2.5mm_P7.62mm_Horizontal
- R29: renamed from R33; footprint (none) -> Resistor_THT:R_Axial_DIN0207_L6.3mm_D2.5mm_P7.62mm_Horizontal
- R30: renamed from R34; footprint (none) -> Resistor_THT:R_Axial_DIN0207_L6.3mm_D2.5mm_P7.62mm_Horizontal
- R31: renamed from R36; footprint (none) -> Resistor_THT:R_Axial_DIN0207_L6.3mm_D2.5mm_P7.62mm_Horizontal
- R32: renamed from R37; footprint (none) -> Resistor_THT:R_Axial_DIN0207_L6.3mm_D2.5mm_P7.62mm_Horizontal
- R42: renamed from R16; value 100K -> 10K
- SW1: footprint (none) -> Button_Switch_THT:SW_PUSH_6mm_H4.3mm
- T1: footprint TDK DCT15EFD-U44S003:TRANS_U44S003_TDK -> oxebots_transformer:TRANS_U44S003_TDK
- U1: footprint cusf:TSSOP-20-EP -> Package_SO:TSSOP-20-1EP_4.4x6.5mm_P0.65mm_EP2.15x3.35mm
- U6: renamed from U8; value AQV453 -> AQV454; footprint RELAY_AQV_DIP6_25X_PAN -> (none)
- renumbered C16 to C13, C17 to C14, C18 to C15, C20 to C18, C21 to C19, C24 to C20, C25 to C21, D4 to D5, PS2 to PS1, Q6 to Q5, Q2 to Q6, Q4 to Q7, R19 to R13, R20 to R16, R21 to R17, R22 to R19, R25 to R21, R26 to R23, R27 to R24, R28 to R25, R13 to R33, R17 to R34, R18 to R35, R14 to R36, R15 to R37, R23 to R44, R24 to R45, U6 to U3, U7 to U5
Connections:
- net +15V_SEC: now also C16.1, C24.1, U2.8 (VCC), U8.8 (V+), U9.2
- net +3.3V: now also J3.1 (Pin_1), J6.1 (Pin_1), J8.1 (Pin_1), J9.1 (Pin_1), U4.16 (VDD), U4.5 (VDDA), U7.4 (V+)
- net EXT_MCU_RX: now also J6.3 (Pin_3)
- net EXT_MCU_TX: now also J6.2 (Pin_2)
- net GND: now also C17.2, J3.2 (Pin_2), J6.4 (Pin_4), J8.5 (Pin_5), J9.8 (Pin_8), U2.3 (C), U4.15 (VSS), U7.11 (V-), U7.3 (+), U7.6 (-), U9.5
- net GNDPWR: now also C16.2, C24.2, D6.2 (A), D7.2 (A2), Q3.3 (S), R20.2, U2.5 (VEE), U8.4 (V-), U8.5 (+), U9.4
- net LT3751_FB: now also U7.13 (-), U7.14; no longer C22.2
- net MCU_OUT_KICK_1: now also R15.1
- net MCU_RST: now also J8.2 (Pin_2)
- net MCU_SWCLK: now also J8.4 (Pin_4)
- net MCU_SWDIO: now also J8.3 (Pin_3)
- net VCAP: now also D4.1 (A1), J5.P
- net at C19.1, R23.2, U5.1: now also R22.2
- net at R37.2, R42.1: now also D7.1 (A1), U8.3 (+)
- net at C22.1: now also R41.1, U7.10 (+), U7.12 (+), U7.7
- net at C18.1, R16.2, U3.1: now also R14.2
- net at R31.1, U6.4: now also D6.1 (K)
- net MCU_IN_DONE renamed EXT_OUT_LT3751_DONE
- net EXT_OUT_LT3751_DONE: now also J9.6 (Pin_6)
- net MCU_IN_FAULT renamed EXT_OUT_LT3751_FAULT
- net EXT_OUT_LT3751_FAULT: now also J9.5 (Pin_5)
- new net: R39.1, U8.6 (-), U9.3
- new net: R40.2, U8.7
- new net: R38.1, RV1.1
- new net: R38.2, U7.2 (-), U9.6
- new net: R39.2, U8.1, U8.2 (-)
- new net: R43.2, RV1.2, RV1.3, U7.1
- new net: Q3.1 (G), R18.2, R20.1
- new net: C22.2, R41.2, R43.1, U7.5 (+)
- new net: D4.2 (A2), J5.N, Q3.2 (D)
- new net: R40.1, U9.1
- new net: C17.1, R15.2, U2.2 (A)
- new net: R18.1, U2.6 (VO), U2.7 (VO)
- new net EXT_IN_LT3751_ENABLE: J9.2 (Pin_2)
- new net EXT_IN_LT3751_KICK_1: J9.3 (Pin_3), R14.1, R22.1
- new net EXT_IN_LT3751_KICK_2: J9.4 (Pin_4)
- new net EXT_OUT_FB: U7.8, U7.9 (-)
- new net EXT_OUT_VSEC_FB: J9.7 (Pin_7)
- no-connect marks 7 -> 6
Other:
- note added: "Feedback Circuit"
- note removed: "Digital Feedback Circuit"
- note removed: "Low-Pass Active Feedback Filter"
- moved on the sheet: C13, C14, C15, C18, C19, C20, C21, D3, D5, J4, J7, JP1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

Commit message: update
Placa parcialmente desenhada, componentes posicionados
Parts:
- removed C11, C8: 220uF, Capacitor_THT:CP_Radial_D8.0mm_P5.00mm, symbol Device:C_US
- removed C17, C18, C19, C20: 100nF, Capacitor_THT:C_Disc_D5.0mm_W2.5mm_P2.50mm, symbol Device:C
- removed C22: C, Capacitor_THT:C_Disc_D5.0mm_W2.5mm_P2.50mm, symbol Device:C
- removed D1: SMBJ26A, Diode_SMD:D_SMB_Handsoldering, symbol Device:D_TVS
- removed D3, D5: 1.5KE300A, Diode_THT:D_DO-201AE_P15.24mm_Horizontal, symbol Diode:1.5KExxA
- removed D7: SMBJ5.0A, Diode_SMD:D_SMB, symbol Diode:SMAJ5.0A
- removed J2: CONN_BUCK, Connector_PinSocket_2.54mm:PinSocket_1x04_P2.54mm_Vertical, symbol Connector:Conn_01x04_Pin
- removed J4, J7: XT30PW-F, oxebots_connectors:AMASS_XT30PW-M, symbol oxebots:XT30PW-F
- removed J6: Conn_01x04, Connector_PinHeader_2.54mm:PinHeader_1x04_P2.54mm_Vertical, symbol Connector_Generic:Conn_01x04
- removed J8: Conn_01x05, Connector_PinHeader_2.54mm:PinHeader_1x05_P2.54mm_Vertical, symbol Connector_Generic:Conn_01x05
- removed JP1: ~, Jumper:SolderJumper-3_P1.3mm_Open_Pad1.0x1.5mm, symbol Jumper:SolderJumper_3_Open
- removed Q2, Q4: CS20N60, Package_TO_SOT_SMD:TO-263-2, symbol Transistor_FET:Q_NMOS_GDS
- removed Q6, Q7: BC547, Package_TO_SOT_THT:TO-92_Inline, symbol Transistor_BJT:BC547
- removed R16, R17, R22: 220R, Resistor_THT:R_Axial_DIN0207_L6.3mm_D2.5mm_P7.62mm_Horizontal, symbol Device:R
- removed R19, R21: 3.3k, Resistor_THT:R_Axial_DIN0207_L6.3mm_D2.5mm_P7.62mm_Horizontal, symbol Device:R
- removed R30: 10k, Resistor_THT:R_Axial_DIN0207_L6.3mm_D2.5mm_P7.62mm_Horizontal, symbol Device:R
- removed R41, R43: R, Resistor_THT:R_Axial_DIN0207_L6.3mm_D2.5mm_P7.62mm_Horizontal, symbol Device:R
- removed SW1: SW_Push, Button_Switch_THT:SW_PUSH_6mm_H4.3mm, symbol Switch:SW_Push
- removed U3, U5: PC817, Package_DIP:DIP-4_W7.62mm, symbol Isolator:PC817
- removed U4: STM32F030F4Px, Package_SO:TSSOP-20_4.4x6.5mm_P0.65mm, symbol MCU_ST_STM32F0:STM32F030F4Px
- removed unit 3 of U7
- removed unit 1 of U7
- removed unit 2 of U7
- removed unit 4 of U7
- added C3, C6: 100nF, Capacitor_SMD:C_0805_2012Metric_Pad1.18x1.45mm_HandSolder, symbol Device:C
- added D4: SMBJ26A, Diode_SMD:D_SMB, symbol Diode:SMAJ26A
- added J3: Conn_01x02, Connector_JST:JST_XH_B2B-XH-A_1x02_P2.50mm_Vertical, symbol Connector_Generic:Conn_01x02
- added Q1, Q2: BC847, Package_TO_SOT_SMD:SOT-23, symbol Transistor_BJT:BC847
- added R10: 1.2k, Resistor_SMD:R_0805_2012Metric_Pad1.20x1.40mm_HandSolder, symbol Device:R
- added R11: 9.1k, Resistor_SMD:R_0805_2012Metric_Pad1.20x1.40mm_HandSolder, symbol Device:R
- added R12, R8, R9: 10k, Resistor_SMD:R_0805_2012Metric_Pad1.20x1.40mm_HandSolder, symbol Device:R
- added R27: 5.6k, Resistor_SMD:R_0805_2012Metric_Pad1.20x1.40mm_HandSolder, symbol Device:R
- added R28, R5: 1k, Resistor_SMD:R_0805_2012Metric_Pad1.20x1.40mm_HandSolder, symbol Device:R
- added RV1: 100k, Potentiometer_THT:Potentiometer_Bourns_3296W_Vertical, symbol Device:R_Potentiometer_Trim
- added unit 3 of U1
- added unit 1 of U1
- added unit 2 of U1
- added unit 4 of U1
- added U2: LMV358, Package_SO:SOIC-8_5.3x6.2mm_P1.27mm, symbol Amplifier_Operational:LM358
- added U3: TLV431DBZ, Package_TO_SOT_SMD:SOT-23, symbol Reference_Voltage:TL431DBZ
- C13: renamed from C16; footprint Capacitor_THT:C_Disc_D5.0mm_W2.5mm_P2.50mm -> Capacitor_SMD:C_0805_2012Metric_Pad1.18x1.45mm_HandSolder
- C19: renamed from C24; footprint Capacitor_THT:C_Rect_L19.0mm_W6.0mm_P15.00mm_MKS4 -> Capacitor_SMD:C_0805_2012Metric_Pad1.18x1.45mm_HandSolder
- C2: renamed from C12; footprint Capacitor_THT:C_Disc_D5.0mm_W2.5mm_P2.50mm -> Capacitor_SMD:C_0805_2012Metric_Pad1.18x1.45mm_HandSolder
- C5: renamed from C23; footprint Capacitor_THT:C_Rect_L19.0mm_W6.0mm_P15.00mm_MKS4 -> Capacitor_SMD:C_0805_2012Metric_Pad1.18x1.45mm_HandSolder
- C7: renamed from C1; footprint Capacitor_THT:C_Disc_D5.0mm_W2.5mm_P2.50mm -> Capacitor_SMD:C_0805_2012Metric_Pad1.18x1.45mm_HandSolder
- C9: value 100nF -> 1nF; footprint Capacitor_THT:C_Disc_D5.0mm_W2.5mm_P2.50mm -> Capacitor_SMD:C_0805_2012Metric_Pad1.18x1.45mm_HandSolder
- D2: renamed from D6; footprint Diode_THT:D_DO-41_SOD81_P10.16mm_Horizontal -> Diode_THT:D_DO-41_SOD81_P7.62mm_Horizontal
- D3: renamed from D4; value 1.5KE300A -> 1.5KE220A
- F1: value 10A -> Fuse
- Q5: renamed from Q3; value FQD20N60 -> FQPF20N60; footprint Package_TO_SOT_SMD:TO-263-2 -> Package_TO_SOT_THT:TO-220F-3_Vertical
- R1: renamed from R9; footprint Resistor_THT:R_Axial_DIN0207_L6.3mm_D2.5mm_P7.62mm_Horizontal -> Resistor_SMD:R_0805_2012Metric_Pad1.20x1.40mm_HandSolder
- R13: value 3.3k -> 10k; footprint Resistor_THT:R_Axial_DIN0207_L6.3mm_D2.5mm_P7.62mm_Horizontal -> Resistor_SMD:R_0805_2012Metric_Pad1.20x1.40mm_HandSolder
- R14, R23: value 220R -> 1k; footprint Resistor_THT:R_Axial_DIN0207_L6.3mm_D2.5mm_P7.62mm_Horizontal -> Resistor_SMD:R_0805_2012Metric_Pad1.20x1.40mm_HandSolder
- R15: renamed from R8; footprint Resistor_THT:R_Axial_DIN0207_L6.3mm_D2.5mm_P7.62mm_Horizontal -> Resistor_SMD:R_0805_2012Metric_Pad1.20x1.40mm_HandSolder
- R16: renamed from R34; footprint Resistor_THT:R_Axial_DIN0207_L6.3mm_D2.5mm_P7.62mm_Horizontal -> Resistor_SMD:R_0805_2012Metric_Pad1.20x1.40mm_HandSolder
- R17: renamed from R44; footprint Resistor_THT:R_Axial_DIN0207_L6.3mm_D2.5mm_P7.62mm_Horizontal -> Resistor_SMD:R_0805_2012Metric_Pad1.20x1.40mm_HandSolder
- R18: renamed from R2; footprint Resistor_THT:R_Axial_DIN0207_L6.3mm_D2.5mm_P7.62mm_Horizontal -> Resistor_SMD:R_0805_2012Metric_Pad1.20x1.40mm_HandSolder
- R19: renamed from R3; footprint Resistor_THT:R_Axial_DIN0207_L6.3mm_D2.5mm_P7.62mm_Horizontal -> Resistor_SMD:R_0805_2012Metric_Pad1.20x1.40mm_HandSolder
- R2: renamed from R11; footprint Resistor_THT:R_Axial_DIN0207_L6.3mm_D2.5mm_P7.62mm_Horizontal -> Resistor_SMD:R_0805_2012Metric_Pad1.20x1.40mm_HandSolder
- R20: renamed from R5; footprint Resistor_THT:R_Axial_DIN0207_L6.3mm_D2.5mm_P7.62mm_Horizontal -> Resistor_SMD:R_0805_2012Metric_Pad1.20x1.40mm_HandSolder
- R21: renamed from R35; footprint Resistor_THT:R_Axial_DIN0207_L6.3mm_D2.5mm_P7.62mm_Horizontal -> Resistor_SMD:R_0805_2012Metric_Pad1.20x1.40mm_HandSolder
- R22: renamed from R45; footprint Resistor_THT:R_Axial_DIN0207_L6.3mm_D2.5mm_P7.62mm_Horizontal -> Resistor_SMD:R_0805_2012Metric_Pad1.20x1.40mm_HandSolder
- R24: value 220R -> 330R; footprint Resistor_THT:R_Axial_DIN0207_L6.3mm_D2.5mm_P7.62mm_Horizontal -> Resistor_SMD:R_0805_2012Metric_Pad1.20x1.40mm_HandSolder
- R25: value 3.3k -> 20k; footprint Resistor_THT:R_Axial_DIN0207_L6.3mm_D2.5mm_P7.62mm_Horizontal -> Resistor_SMD:R_0805_2012Metric_Pad1.20x1.40mm_HandSolder
- R26, R7: footprint Resistor_THT:R_Axial_DIN0207_L6.3mm_D2.5mm_P7.62mm_Horizontal -> Resistor_SMD:R_0805_2012Metric_Pad1.20x1.40mm_HandSolder
- R3: renamed from R10; footprint Resistor_THT:R_Axial_DIN0207_L6.3mm_D2.5mm_P7.62mm_Horizontal -> Resistor_SMD:R_0805_2012Metric_Pad1.20x1.40mm_HandSolder
- R31: renamed from R38; value 27k -> 270k; footprint Resistor_THT:R_Axial_DIN0207_L6.3mm_D2.5mm_P7.62mm_Horizontal -> Resistor_SMD:R_0805_2012Metric_Pad1.20x1.40mm_HandSolder
- R32: renamed from R27; value 470R -> 1k; footprint Resistor_THT:R_Axial_DIN0207_L6.3mm_D2.5mm_P7.62mm_Horizontal -> Resistor_SMD:R_0805_2012Metric_Pad1.20x1.40mm_HandSolder
- R33: renamed from R15; footprint Resistor_THT:R_Axial_DIN0207_L6.3mm_D2.5mm_P7.62mm_Horizontal -> Resistor_SMD:R_0805_2012Metric_Pad1.20x1.40mm_HandSolder
- R36: renamed from R40; value 470R -> 1k; footprint Resistor_THT:R_Axial_DIN0207_L6.3mm_D2.5mm_P7.62mm_Horizontal -> Resistor_SMD:R_0805_2012Metric_Pad1.20x1.40mm_HandSolder
- R38: renamed from R18; footprint Resistor_THT:R_Axial_DIN0207_L6.3mm_D2.5mm_P7.62mm_Horizontal -> Resistor_SMD:R_0805_2012Metric_Pad1.20x1.40mm_HandSolder
- R39: renamed from R29; footprint Resistor_THT:R_Axial_DIN0207_L6.3mm_D2.5mm_P7.62mm_Horizontal -> oxebots:Resistor_RX24_10W
- R4: renamed from R12; footprint Resistor_THT:R_Axial_DIN0207_L6.3mm_D2.5mm_P7.62mm_Horizontal -> Resistor_SMD:R_0805_2012Metric_Pad1.20x1.40mm_HandSolder
- R40: renamed from R20; footprint Resistor_THT:R_Axial_DIN0207_L6.3mm_D2.5mm_P7.62mm_Horizontal -> Resistor_SMD:R_0805_2012Metric_Pad1.20x1.40mm_HandSolder
- R41: renamed from R39; value 47k -> 330k; footprint Resistor_THT:R_Axial_DIN0207_L6.3mm_D2.5mm_P7.62mm_Horizontal -> Resistor_SMD:R_0805_2012Metric_Pad1.20x1.40mm_HandSolder
- R42: renamed from R33; value 330k -> 510k; footprint Resistor_THT:R_Axial_DIN0207_L6.3mm_D2.5mm_P7.62mm_Horizontal -> Resistor_THT:R_Axial_DIN0207_L6.3mm_D2.5mm_P15.24mm_Horizontal
- R43: renamed from R36; value 330k -> 510k
- R44: renamed from R37; value 330k -> 47k
- R45: renamed from R42; value 10K -> 33k
- R6: renamed from R4; footprint Resistor_THT:R_Axial_DIN0207_L6.3mm_D2.5mm_P7.62mm_Horizontal -> Resistor_SMD:R_0805_2012Metric_Pad1.20x1.40mm_HandSolder
- U1: renamed from U7; value LMF324 -> LM324; footprint (none) -> Package_SO:SOIC-14_3.9x8.7mm_P1.27mm
- U5: renamed from U6; footprint (none) -> Package_DIP:DIP-6_W7.62mm_LongPads
- U6: renamed from U9; footprint Package_DIP:DIP-8_W7.62mm_LongPads -> Package_DIP:DIP-8_W10.16mm_LongPads
- U7: renamed from U2; footprint Package_DIP:DIP-8_W7.62mm -> Package_DIP:DIP-8_W7.62mm_LongPads
- U8: footprint Package_DIP:DIP-8_W7.62mm -> Package_SO:SOIC-8_5.3x6.2mm_P1.27mm
- renumbered C2 to C1, C13 to C10, C7 to C11, C4 to C12, C21 to C15, C5 to C16, C15 to C17, C6 to C18, C3 to C4, C10 to C8, D2 to D1, J3 to J2, J9 to J4, Q1 to Q3, Q5 to Q4, R6 to R29, R1 to R30, R28 to R34, R31 to R35, R32 to R37, RV1 to RV2, U1 to U4
Connections:
- net EXT_IN_LT3751_KICK_2 is gone; now on net EXT_OUT_LT3751_FAULT: J4.4 (Pin_4)
- net EXT_OUT_VSEC_FB is gone; now on net GND: J4.7 (Pin_7)
- net MCU_OUT_BLEEDER is gone; now on net +12V: R32.1
- net MCU_OUT_ENABLE is gone; now on net EXT_IN_LT3751_ENABLE: R7.1
- net MCU_OUT_KICK_1 is gone; now on net EXT_IN_LT3751_KICK_1: R33.1
- net MCU_OUT_KICK_2 is gone; now on an unnamed net: R23.1
- net MCU_RST is gone; now on net GND: R26.2
- net OVLO_1 is gone; now on net LT3751_OVLO_1: R2.2
- net OVLO_2 is gone; now on net LT3751_OVLO_2: R4.2
- net UVLO_1 is gone; now on net LT3751_UVLO_1: R1.2
- net UVLO_2 is gone; now on net LT3751_UVLO_2: R3.2
- net +12V: now also C5.1, U1.4 (V+), C3.1, J3.1 (Pin_1); no longer C9.1
- net +15V_SEC: no longer R13.1
- net +24V: now also D4.1 (A1)
- net +3.3V: now also C6.1, R27.1, U2.8 (V+); no longer C5.1, R26.1, U1.4 (V+)
- net EXT_IN_LT3751_ENABLE: now also J4.6 (Pin_6); no longer J4.2 (Pin_2)
- net EXT_IN_LT3751_KICK_1: now also J4.2 (Pin_2); no longer J4.3 (Pin_3), R14.1
- net EXT_OUT_FB: now also J4.3 (Pin_3), R5.1
- net EXT_OUT_LT3751_DONE: now also J4.5 (Pin_5), Q1.3 (C); no longer J4.6 (Pin_6)
- net EXT_OUT_LT3751_FAULT: now also Q2.3 (C); no longer J4.5 (Pin_5)
- net GND: now also R24.2, C3.2, C6.2, D4.2 (A2), J3.2 (Pin_2), Q1.2 (E), Q2.2 (E), R11.2, R28.2, R9.2, U1.10 (+), U2.4 (V-), U3.3 (A); no longer C9.2
- net GNDPWR: now also U8.3 (+); no longer R25.2, U8.5 (+)
- net LT3751_DONE: now also Q1.1 (B)
- net LT3751_FAULT: now also Q2.1 (B)
- net LT3751_FB: now also R14.1, R10.1, U3.1 (K)
- net at R23.2: now also RV1.1, U1.3 (+)
- net at R44.2, R45.1: now also U8.5 (+); no longer U8.3 (+)
- net at R41.1, U6.3: now also U8.2 (-); no longer U8.6 (-)
- net at U8.7: now also R41.2, U8.6 (-); no longer R36.2
- net at R31.2, U6.6: now also C9.1, U1.9 (-)
- net at R14.2: now also U1.1, U1.2 (-)
- net at R24.1: now also RV1.2, RV1.3
- net at R25.1: now also U1.6 (-), U1.7; no longer R24.2
- net at RV2.2, RV2.3: now also C9.2, U1.5 (+), U1.8
- net at R13.2: now also U2.6 (-), U2.7
- new net: R36.2, U8.1
- new net: R10.2, R11.1, U3.2 (REF)
- new net: R5.2, R8.1, U2.1
- new net: R8.2, R9.1, U2.2 (-)
- new net: R12.1, R13.1, U2.3 (+)
- new net: R25.2, R26.1, U1.12 (+)
- new net: R27.2, R28.1, U2.5 (+)
- new net: R12.2, U1.13 (-), U1.14
- no-connect marks 6 -> 4
Other:
- note removed: "External Programmer (ST Link)"
- note removed: "External UART"
- note removed: "Microcontroller STM32"
- moved on the sheet: C10, C13, C14, C15, C17, C19, C5, D2, D3, J5, PS1, Q4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
