File: pcbs/kicker/interfacecircuito.kicad_pcb (KiCad board)
At the start: 2 copper layers, 117.9 x 140 mm, 70 parts, among them J1 Conn_01x02, J5 Conn_02x08_Odd_Even, Q1 IRFB3077, Q2 IRFB3077, Q3 BC338, U2 IR2101, U3 PC817, U4 LM358, U5 LM324

Commit message: Resolução de Warnings do esquemático, substituição de conectores on/off e conector de solenoide
Parts:
- removed C8: 100nF, Capacitor_SMD:C_0805_2012Metric_Pad1.18x1.45mm_HandSolder
- removed R22, R23: 12k 2W, Resistor_THT:R_Axial_DIN0617_L17.0mm_D6.0mm_P20.32mm_Horizontal
- added J2: XT30PW-M, oxebots:AMASS_XT30PW-M, F.Cu at (109.0, 114.0)
- D4, D6: footprint LED_SMD:LED_0805_2012Metric_Pad1.15x1.40mm_HandSolder -> LED_THT:LED_D5.0mm
- J1: footprint Connector_PinHeader_1.00mm:PinHeader_1x02_P1.00mm_Vertical -> Connector_JST:JST_EH_B2B-EH-A_1x02_P2.50mm_Vertical
- R25: value 10k -> 1k
- TP4: moved to B.Cu
- moved D4 75.2 mm to (56.7, 80.0), turned to 0 degrees
- moved R12 12.6 mm to (131.0, 131.6), turned to 90 degrees
- moved TP4 10.5 mm to (131.0, 118.0), turned to 180 degrees
- moved TP7 5.32 mm to (67.5, 89.0)
- moved C11 5.02 mm to (142.0, 62.0)
- moved D6 3.74 mm to (124.5, 108.8), turned to 90 degrees
- moved JP2 3.65 mm to (64.0, 99.5)
- moved C13 3.35 mm to (133.1, 81.0)
- moved R25 3.00 mm to (123.0, 90.4)
- moved Q3 2.55 mm to (59.4, 100.7), turned to -90 degrees
- moved R2 2.50 mm to (144.5, 102.2)
- moved R3 2.06 mm to (131.5, 109.6)
- moved D2 1.00 mm to (136.1, 90.5)
- moved J1 0.84 mm to (123.7, 70.2), turned to 90 degrees
- moved C1 0.79 mm to (137.8, 87.2), turned to 0 degrees
Connections:
- D4 pad 1: HV - -> Net-(D4-K)
- D4 pad 2: Net-(D4-A) -> OUT_SIGNAL_HV
- Q3 pad 1: unconnected-(Q3-C-Pad1) -> Net-(D4-K)
- Q3 pad 2: unconnected-(Q3-B-Pad2) -> Net-(Q3-B)
- Q3 pad 3: unconnected-(Q3-E-Pad3) -> HV -
- U4 pad 6: Net-(U4B--) -> Net-(Q3-B)
- U4 pad 7: Net-(U4B--) -> Net-(Q3-B)
Routing:
- net SOLENOID +: track 1.44 -> 50.1 mm
- net SOLENOID -: track 23.6 -> 54.3 mm
- net Net-(D4-K): track 0.00 -> 29.3 mm, vias 0 -> 2
- net GND: track 104.7 -> 130.6 mm
- net Net-(Q3-B): track 0.00 -> 21.9 mm
- net (no net): track 21.9 -> 0.00 mm
- net V_BAT: track 26.2 -> 45.6 mm
- net Net-(R14-Pad2): track 57.3 -> 40.4 mm
- net OUT_SIGNAL_HV: track 42.4 -> 34.3 mm
- net Net-(Q2-G): track 4.14 -> 11.9 mm
- net Net-(R22-Pad2): track 7.57 -> 0.00 mm
- net GATE_BLEED: track 34.5 -> 27.5 mm, vias 1 -> 2
- net HV +: track 50.6 -> 44.0 mm
- net V_SHUNT: track 172.9 -> 178.7 mm
- net HV -: track 7.76 -> 12.1 mm, vias 1 -> 116
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- removed copper zone on F.Cu, net (none)

Commit message: Resolução de EDR Mudança nas trilhas de 24V mudança do footprint dos capacitores bulk
Parts:
- added G***: LOGO, oxebots:Icon_High_Voltage_10mm, F.Cu at (144.2, 71.2)
- C2, C5: footprint Capacitor_THT:C_Radial_D18.0mm_H35.5mm_P7.50mm -> Capacitor_THT:CP_Radial_D30.0mm_P10.00mm_SnapIn
- moved C2 2.63 mm to (150.0, 43.0)
- moved C4 2.23 mm to (137.0, 59.2)
- moved C5 1.30 mm to (150.2, 157.0)
Routing:
- net +24V: track 119.3 -> 7.25 mm
- net GND: track 130.6 -> 57.7 mm, vias 0 -> 120
- net V_BAT: track 45.6 -> 19.4 mm
- added copper zone on B.Cu, net +24V
- added copper zone on F.Cu, net +24V
Other:
- board text added: "Cuidado Alta Tensão"

Commit message: mudança na posição do conector da solenoide
Parts:
- added G***: LOGO, oxebots:Icon_High_Voltage_10mm, F.Cu at (145.8, 107.2)
- moved R12 6.16 mm to (125.7, 128.5), turned to 0 degrees
- moved G*** 5.78 mm to (146.0, 76.8)
- moved J2 3.50 mm to (105.8, 112.7)
- moved TP4 2.06 mm to (130.5, 116.0)
- moved R13 1.52 mm to (117.5, 136.0)
- moved Q2 0.53 mm to (120.8, 127.5)
Routing:
- net GATE_BLEED: track 27.5 -> 36.5 mm
- net Net-(Q2-G): track 11.9 -> 7.04 mm
- net SOLENOID -: track 54.3 -> 58.0 mm
- net SOLENOID +: track 50.1 -> 53.1 mm
- net Net-(Q2-D): track 9.62 -> 8.79 mm
- net HV +: track 44.0 -> 43.3 mm
