File: pcbs/main/pcbs/main/motors.kicad_sch (KiCad schematic)
At the start: 50 parts, among them U1 4052, U2 74HC595

Commit message: alteração de layout utilizado em teste para calibração dos encoders AS5600 implementando comunicação no barramento I2C
Parts:
- removed U2: 74HC595, Package_DIP:DIP-16_W7.62mm, symbol 74xx:74HC595
- M1, M2, M3, M4: renamed from M?; value ~ -> (none)
- gave numbers to parts that had none: 44
Connections:
- net GND: now also U1.6 (Inh)
- net MUX_A: now reaches U1.10 (A)
- net MUX_B: now reaches U1.9 (B)
